File: kicad/beat707/beat707.kicad_pcb (KiCad board)
At the start: 2 copper layers, 230 x 130 mm, 59 parts, among them J1 USB_B, J2 DIN-5_180degree, J3 AudioJack3_Ground, J4 DIN-5_180degree, SW1 SW_Push, SW10 SW_Push, SW11 SW_Push, SW12 SW_Push, SW13 SW_Push, SW14 SW_Push, SW15 SW_Push, SW16 SW_Push, SW17 SW_Push, SW18 SW_Push, SW19 SW_Push, SW2 SW_Push, SW20 SW_Push, SW21 SW_Push, SW22 SW_Push, SW23 SW_Push, SW24 SW_Push, SW3 SW_Push, SW4 SW_Push, SW5 SW_Push, SW6 SW_Push, SW7 SW_Push, SW8 SW_Push, SW9 SW_Push, U1 ATmega328-PU, U2 CA56-12EWA, U3 CA56-12EWA, U4 CA56-12EWA, U5 CA56-12EWA, U6 CA56-12EWA, U7 CA56-12EWA

Commit message: 3 new buttons and a rotary encoder (ALPS EC12E)
Parts:
- added SW25: SW_Push, beat707:K2-1103SP-A4SW-04, F.Cu at (59.7, 148.6)
- added SW26: SW_Push, beat707:K2-1103SP-A4SW-04, F.Cu at (59.7, 166.4)
- added SW27: SW_Push, beat707:K2-1103SP-A4SW-04, F.Cu at (59.7, 185.4)
- added SW28: Rotary_Encoder, Rotary_Encoder:RotaryEncoder_Alps_EC12E_Vertical_H20mm, F.Cu at (306.1, 138.4)
- moved D1 236.0 mm to (351.8, 75.4)
- moved D2 224.8 mm to (351.8, 79.9)
- moved D3 217.3 mm to (356.7, 75.4)
- moved D4 204.8 mm to (356.7, 79.9)
- moved SW4 191.3 mm to (344.2, 151.1)
- moved SW5 182.8 mm to (326.4, 189.2)
- moved SW3 167.5 mm to (306.1, 149.9)
- moved U2 150.5 mm to (251.5, 144.8)
- moved SW8 138.8 mm to (326.4, 168.9)
- moved D5 134.7 mm to (288.3, 120.7)
- moved D6 125.9 mm to (288.3, 124.5)
- moved U1 121.7 mm to (170.2, 106.7)
- moved U3 116.5 mm to (99.1, 144.8)
- moved D7 114.8 mm to (288.3, 128.3)
- moved D8 105.7 mm to (288.3, 132.1)
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Other:
- board size 230 x 130 mm -> 292.1 x 134.6 mm

Commit message: all LEDs changed to through-hole, 3mm
Parts:
- D1, D10, D11, D12, D13, D14, D15, D16, D17, D18, D19, D2, D20, D21, D22, D23, D24, D3, D4, D5, D6, D7, D8, D9: footprint LED_SMD:LED_0603_1608Metric_Castellated -> LED_THT:LED_D3.0mm

Commit message: new version from Gert with changed positions
Parts:
- removed D1, D2, D3, D4: LED, LED_THT:LED_D3.0mm
- moved SW5 246.6 mm to (81.3, 162.6)
- moved SW8 246.1 mm to (81.3, 190.5)
- moved SW26 227.9 mm to (287.1, 181.6), turned to 270 degrees
- moved SW6 167.1 mm to (320.0, 172.7)
- moved SW25 137.8 mm to (195.6, 125.8), turned to 270 degrees
- moved SW27 56.0 mm to (55.9, 129.5), turned to 270 degrees
- moved SW2 44.4 mm to (170.2, 139.7)
- moved SW1 43.3 mm to (152.4, 137.2)
- moved D8 40.7 mm to (289.6, 172.7)
- moved D7 39.4 mm to (289.6, 167.6)
- moved D6 38.1 mm to (289.6, 162.6)
- moved D5 36.9 mm to (289.6, 157.5)
- moved SW3 22.5 mm to (322.6, 134.6)
- moved SW4 21.8 mm to (322.5, 153.4)
- moved SW28 18.8 mm to (289.6, 147.3), turned to 90 degrees
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