File: kicad/beat707/beat707.kicad_pcb (KiCad board)
At the start: 2 copper layers, 292.1 x 134.6 mm, 59 parts, among them J1 USB_B, J2 DIN-5_180degree, J3 AudioJack3_Ground, J4 DIN-5_180degree, SW1 SW_Push, SW10 SW_Push, SW11 SW_Push, SW12 SW_Push, SW13 SW_Push, SW14 SW_Push, SW15 SW_Push, SW16 SW_Push, SW17 SW_Push, SW18 SW_Push, SW19 SW_Push, SW2 SW_Push, SW20 SW_Push, SW21 SW_Push, SW22 SW_Push, SW23 SW_Push, SW24 SW_Push, SW25 SW_Push, SW26 SW_Push, SW27 SW_Push, SW28 Rotary_Encoder, SW3 SW_Push, SW4 SW_Push, SW5 SW_Push, SW6 SW_Push, SW7 SW_Push, SW8 SW_Push, SW9 SW_Push, U1 ATmega328-PU, U2 CA56-12EWA, U3 CA56-12EWA, U4 CA56-12EWA, U5 CA56-12EWA, U6 CA56-12EWA, U7 CA56-12EWA

Commit message: final UI layout +silkscreen
basic silkscreen, more to come
Parts:
- moved SW3 3.81 mm to (87.6, 190.5)
- moved SW4 3.81 mm to (311.1, 190.5)
- moved SW5 3.81 mm to (323.9, 190.5)
- moved SW8 3.81 mm to (74.9, 190.5)
- moved SW27 1.27 mm to (55.9, 158.8)
Other:
- board text added: "BANK"
- board text added: "MUTE"
- board text added: "PATTERN"
- board text added: "PLAY RECORD"
- board text added: "SHIFT"
- board text added: "STOP"
- board text added: "TRACK"
- board text added: "VAL+"
- board text added: "VAL-"
- board text added: "VARIATION"
- board text added: "VELOCITY"
Changed lines of the file:
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@@
   (general
     (thickness 1.6)
-    (drawings 4)
+    (drawings 15)
     (tracks 0)
     (zones 0)
@@
   )
   (module beat707:K2-1103SP-A4SW-04 (layer F.Cu)
-    (at 87.55 186.69 90)
+    (at 87.63 190.5 90)
     (descr "4 digit 7 segment green LED, http://www.kingbrightusa.com/images/catalog/SPEC/CA56-12EWA.pdf")
     (tags "4 digit 7 segment green LED")
@@
   )
   (module beat707:K2-1103SP-A4SW-04 (layer F.Cu)
-    (at 311.15 186.69 90)
+    (at 311.15 190.5 90)
     (descr "4 digit 7 segment green LED, http://www.kingbrightusa.com/images/catalog/SPEC/CA56-12EWA.pdf")
     (tags "4 digit 7 segment green LED")
@@
   )
   (module beat707:K2-1103SP-A4SW-04 (layer F.Cu)
-    (at 323.85 186.69 90)
+    (at 323.85 190.5 90)
     (descr "4 digit 7 segment green LED, http://www.kingbrightusa.com/images/catalog/SPEC/CA56-12EWA.pdf")
     (tags "4 digit 7 segment green LED")
@@
   )
   (module beat707:K2-1103SP-A4SW-04 (layer F.Cu)
-    (at 74.93 186.69 90)
+    (at 74.93 190.5 90)
     (descr "4 digit 7 segment green LED, http://www.kingbrightusa.com/images/catalog/SPEC/CA56-12EWA.pdf")
     (tags "4 digit 7 segment green LED")
@@
   )
   (module beat707:K2-1103SP-A4SW-04 (layer F.Cu)
-    (at 55.88 157.48 270)
+    (at 55.88 158.75 270)
     (descr "4 digit 7 segment green LED, http://www.kingbrightusa.com/images/catalog/SPEC/CA56-12EWA.pdf")
     (tags "4 digit 7 segment green LED")
@@
     )
   )
+  (gr_text VAL+ (at 311.15 175.26) (layer F.SilkS)
+    (effects (font (size 1.5 1.5) (thickness 0.3)))
+  )
+  (gr_text "VAL-\n" (at 298.45 175.26) (layer F.SilkS)
+    (effects (font (size 1.5 1.5) (thickness 0.3)))
+  )
+  (gr_text VELOCITY (at 74.93 175.26) (layer F.SilkS)
+    (effects (font (size 1.5 1.5) (thickness 0.3)))
+  )
+  (gr_text "TRACK\n" (at 62.23 175.26) (layer F.SilkS)
+    (effects (font (size 1.5 1.5) (thickness 0.3)))
+  )
+  (gr_text "SHIFT\n" (at 68.58 152.4) (layer F.SilkS)
+    (effects (font (size 1.5 1.5) (thickness 0.3)))
+  )
+  (gr_text "VARIATION\n" (at 68.58 129.54) (layer F.SilkS)
+    (effects (font (size 1.5 1.5) (thickness 0.3)))
+  )
+  (gr_text "PATTERN\n" (at 227.33 129.54) (layer F.SilkS)
+    (effects (font (size 1.5 1.5) (thickness 0.3)))
+  )
+  (gr_text "BANK\n" (at 214.63 129.54) (layer F.SilkS)
+    (effects (font (size 1.5 1.5) (thickness 0.3)))
+  )
+  (gr_text MUTE (at 186.69 129.54) (layer F.SilkS)
+    (effects (font (size 1.5 1.5) (thickness 0.3)))
+  )
+  (gr_text STOP (at 158.75 129.54) (layer F.SilkS)
+    (effects (font (size 1.5 1.5) (thickness 0.3)))
+  )
+  (gr_text "PLAY\nRECORD" (at 146.05 128.27) (layer F.SilkS)
+    (effects (font (size 1.5 1.5) (thickness 0.3)))
+  )
   (gr_line (start 50.8 203.2) (end 50.8 68.58) (angle 90) (layer Edge.Cuts) (width 0.15))

Commit message: more LEDs, switches and resistors for version encoding
Parts:
- added C1: 100nF, Capacitor_SMD:C_0805_2012Metric, F.Cu at (384.0, 137.2)
- added C2: 10uF, Capacitor_SMD:C_0805_2012Metric, F.Cu at (387.4, 137.2)
- added C3: 100nF, Capacitor_SMD:C_0805_2012Metric, F.Cu at (358.1, 210.5)
- added C4: 10uF, Capacitor_SMD:C_0805_2012Metric, F.Cu at (354.7, 210.5)
- added C5: 100nF, Capacitor_SMD:C_0805_2012Metric, F.Cu at (515.3, 137.2)
- added C6: 10uF, Capacitor_SMD:C_0805_2012Metric, F.Cu at (511.9, 137.2)
- added D1: LED, LED_THT:LED_D3.0mm, F.Cu at (443.5, 118.8)
- added D10: 1N4148, Diode_THT:D_DO-35_SOD27_P7.62mm_Horizontal, F.Cu at (383.4, 126.8)
- added D100: LED, LED_THT:LED_D3.0mm, F.Cu at (566.5, 118.3)
- added D101: 1N4148, Diode_THT:D_DO-35_SOD27_P7.62mm_Horizontal, F.Cu at (585.9, 97.1)
- added D102: 1N4148, Diode_THT:D_DO-35_SOD27_P7.62mm_Horizontal, F.Cu at (566.4, 108.7)
- added D103: 1N4148, Diode_THT:D_DO-35_SOD27_P7.62mm_Horizontal, F.Cu at (550.4, 131.9)
- added D104: 1N4148, Diode_THT:D_DO-35_SOD27_P7.62mm_Horizontal, F.Cu at (576.1, 105.6)
- added D105: 1N4148, Diode_THT:D_DO-35_SOD27_P7.62mm_Horizontal, F.Cu at (540.6, 129.9)
- added D106: 1N4148, Diode_THT:D_DO-35_SOD27_P7.62mm_Horizontal, F.Cu at (576.1, 91.8)
- added D107: 1N4148, Diode_THT:D_DO-35_SOD27_P7.62mm_Horizontal, F.Cu at (576.1, 94.4)
- added D108: 1N4148, Diode_THT:D_DO-35_SOD27_P7.62mm_Horizontal, F.Cu at (566.4, 106.1)
- added D109: 1N4148, Diode_THT:D_DO-35_SOD27_P7.62mm_Horizontal, F.Cu at (566.4, 100.5)
- added D11: 1N4148, Diode_THT:D_DO-35_SOD27_P7.62mm_Horizontal, F.Cu at (373.6, 134.5)
- added D110: 1N4148, Diode_THT:D_DO-35_SOD27_P7.62mm_Horizontal, F.Cu at (585.9, 94.5)
- added D111: 1N4148, Diode_THT:D_DO-35_SOD27_P7.62mm_Horizontal, F.Cu at (540.6, 132.4)
- added D112: 1N4148, Diode_THT:D_DO-35_SOD27_P7.62mm_Horizontal, F.Cu at (595.2, 78.9)
- added D113: 1N4148, Diode_THT:D_DO-35_SOD27_P7.62mm_Horizontal, F.Cu at (550.4, 129.4)
- added D114: 1N4148, Diode_THT:D_DO-35_SOD27_P7.62mm_Horizontal, F.Cu at (511.3, 131.9)
- added D115: 1N4148, Diode_THT:D_DO-35_SOD27_P7.62mm_Horizontal, F.Cu at (511.3, 129.4)
- added D116: 1N4148, Diode_THT:D_DO-35_SOD27_P7.62mm_Horizontal, F.Cu at (521.0, 126.8)
- added D117: 1N4148, Diode_THT:D_DO-35_SOD27_P7.62mm_Horizontal, F.Cu at (566.4, 88.8)
- added D118: 1N4148, Diode_THT:D_DO-35_SOD27_P7.62mm_Horizontal, F.Cu at (511.3, 126.8)
- added D119: 1N4148, Diode_THT:D_DO-35_SOD27_P7.62mm_Horizontal, F.Cu at (501.5, 135.5)
- added D12: 1N4148, Diode_THT:D_DO-35_SOD27_P7.62mm_Horizontal, F.Cu at (373.6, 131.9)
- added D120: 1N4148, Diode_THT:D_DO-35_SOD27_P7.62mm_Horizontal, F.Cu at (501.5, 132.9)
- added D13: LED, LED_THT:LED_D3.0mm, F.Cu at (438.6, 118.8)
- added D14: LED, LED_THT:LED_D3.0mm, F.Cu at (432.3, 127.8)
- added D15: LED, LED_THT:LED_D3.0mm, F.Cu at (458.1, 98.6)
- added D16: LED, LED_THT:LED_D3.0mm, F.Cu at (448.3, 107.6)
- added D17: LED, LED_THT:LED_D3.0mm, F.Cu at (438.6, 123.3)
- added D18: LED, LED_THT:LED_D3.0mm, F.Cu at (463.0, 98.6)
- added D19: LED, LED_THT:LED_D3.0mm, F.Cu at (458.1, 103.1)
- added D2: LED, LED_THT:LED_D3.0mm, F.Cu at (472.8, 89.1)
- added D20: LED, LED_THT:LED_D3.0mm, F.Cu at (448.3, 112.2)
- added D21: 1N4148, Diode_THT:D_DO-35_SOD27_P7.62mm_Horizontal, F.Cu at (363.8, 137.0)
- added D22: 1N4148, Diode_THT:D_DO-35_SOD27_P7.62mm_Horizontal, F.Cu at (363.8, 134.5)
- added D23: 1N4148, Diode_THT:D_DO-35_SOD27_P7.62mm_Horizontal, F.Cu at (373.6, 129.4)
- added D24: 1N4148, Diode_THT:D_DO-35_SOD27_P7.62mm_Horizontal, F.Cu at (373.6, 126.8)
- added D25: 1N4148, Diode_THT:D_DO-35_SOD27_P7.62mm_Horizontal, F.Cu at (402.9, 129.4)
- added D26: 1N4148, Diode_THT:D_DO-35_SOD27_P7.62mm_Horizontal, F.Cu at (383.4, 135.0)
- added D27: 1N4148, Diode_THT:D_DO-35_SOD27_P7.62mm_Horizontal, F.Cu at (393.1, 131.9)
- added D28: 1N4148, Diode_THT:D_DO-35_SOD27_P7.62mm_Horizontal, F.Cu at (393.1, 129.4)
- added D29: 1N4148, Diode_THT:D_DO-35_SOD27_P7.62mm_Horizontal, F.Cu at (363.8, 131.9)
- added D3: LED, LED_THT:LED_D3.0mm, F.Cu at (467.9, 93.6)
- added D30: 1N4148, Diode_THT:D_DO-35_SOD27_P7.62mm_Horizontal, F.Cu at (393.1, 126.8)
- added D31: 1N4148, Diode_THT:D_DO-35_SOD27_P7.62mm_Horizontal, F.Cu at (383.4, 129.4)
- added D32: 1N4148, Diode_THT:D_DO-35_SOD27_P7.62mm_Horizontal, F.Cu at (438.5, 88.8)
- added D33: 1N4148, Diode_THT:D_DO-35_SOD27_P7.62mm_Horizontal, F.Cu at (402.9, 126.8)
- added D34: 1N4148, Diode_THT:D_DO-35_SOD27_P7.62mm_Horizontal, F.Cu at (363.8, 126.8)
- added D35: 1N4148, Diode_THT:D_DO-35_SOD27_P7.62mm_Horizontal, F.Cu at (363.8, 129.4)
- added D36: 1N4148, Diode_THT:D_DO-35_SOD27_P7.62mm_Horizontal, F.Cu at (438.5, 93.9)
- added D37: 1N4148, Diode_THT:D_DO-35_SOD27_P7.62mm_Horizontal, F.Cu at (448.2, 88.8)
- added D38: 1N4148, Diode_THT:D_DO-35_SOD27_P7.62mm_Horizontal, F.Cu at (412.7, 126.8)
- added D39: 1N4148, Diode_THT:D_DO-35_SOD27_P7.62mm_Horizontal, F.Cu at (438.5, 91.3)
- added D4: LED, LED_THT:LED_D3.0mm, F.Cu at (467.9, 89.1)
- added D40: 1N4148, Diode_THT:D_DO-35_SOD27_P7.62mm_Horizontal, F.Cu at (393.1, 134.5)
- added D49: 1N4148, Diode_THT:D_DO-35_SOD27_P7.62mm_Horizontal, F.Cu at (363.8, 205.2)
- added D50: 1N4148, Diode_THT:D_DO-35_SOD27_P7.62mm_Horizontal, F.Cu at (354.1, 208.2)
- added D51: 1N4148, Diode_THT:D_DO-35_SOD27_P7.62mm_Horizontal, F.Cu at (354.1, 205.7)
- added D52: 1N4148, Diode_THT:D_DO-35_SOD27_P7.62mm_Horizontal, F.Cu at (354.1, 203.2)
- added D53: LED, LED_THT:LED_D3.0mm, F.Cu at (472.8, 162.3)
- added D54: LED, LED_THT:LED_D3.0mm, F.Cu at (467.9, 166.9)
- added D55: LED, LED_THT:LED_D3.0mm, F.Cu at (467.9, 162.3)
- added D56: LED, LED_THT:LED_D3.0mm, F.Cu at (448.3, 183.9)
- added D57: LED, LED_THT:LED_D3.0mm, F.Cu at (438.6, 193.1)
- added D58: LED, LED_THT:LED_D3.0mm, F.Cu at (432.3, 201.1)
- added D59: LED, LED_THT:LED_D3.0mm, F.Cu at (422.5, 207.2)
- added D60: LED, LED_THT:LED_D3.0mm, F.Cu at (458.1, 171.3)
- added D61: 1N4148, Diode_THT:D_DO-35_SOD27_P7.62mm_Horizontal, F.Cu at (363.8, 202.7)
- added D62: 1N4148, Diode_THT:D_DO-35_SOD27_P7.62mm_Horizontal, F.Cu at (363.8, 200.1)
- added D63: 1N4148, Diode_THT:D_DO-35_SOD27_P7.62mm_Horizontal, F.Cu at (363.8, 210.3)
- added D64: 1N4148, Diode_THT:D_DO-35_SOD27_P7.62mm_Horizontal, F.Cu at (373.6, 200.1)
- added D65: 1N4148, Diode_THT:D_DO-35_SOD27_P7.62mm_Horizontal, F.Cu at (402.9, 205.2)
- added D66: 1N4148, Diode_THT:D_DO-35_SOD27_P7.62mm_Horizontal, F.Cu at (448.2, 162.1)
- added D67: 1N4148, Diode_THT:D_DO-35_SOD27_P7.62mm_Horizontal, F.Cu at (402.9, 202.7)
- added D68: 1N4148, Diode_THT:D_DO-35_SOD27_P7.62mm_Horizontal, F.Cu at (393.1, 207.8)
- added D69: 1N4148, Diode_THT:D_DO-35_SOD27_P7.62mm_Horizontal, F.Cu at (458.0, 167.8)
- added D70: 1N4148, Diode_THT:D_DO-35_SOD27_P7.62mm_Horizontal, F.Cu at (438.5, 165.1)
- added D71: 1N4148, Diode_THT:D_DO-35_SOD27_P7.62mm_Horizontal, F.Cu at (393.1, 210.3)
- added D72: 1N4148, Diode_THT:D_DO-35_SOD27_P7.62mm_Horizontal, F.Cu at (373.6, 202.7)
- added D73: 1N4148, Diode_THT:D_DO-35_SOD27_P7.62mm_Horizontal, F.Cu at (393.1, 200.1)
- added D74: 1N4148, Diode_THT:D_DO-35_SOD27_P7.62mm_Horizontal, F.Cu at (383.4, 203.2)
- added D75: 1N4148, Diode_THT:D_DO-35_SOD27_P7.62mm_Horizontal, F.Cu at (383.4, 205.7)
- added D76: 1N4148, Diode_THT:D_DO-35_SOD27_P7.62mm_Horizontal, F.Cu at (393.1, 202.7)
- added D77: 1N4148, Diode_THT:D_DO-35_SOD27_P7.62mm_Horizontal, F.Cu at (393.1, 205.2)
- added D78: 1N4148, Diode_THT:D_DO-35_SOD27_P7.62mm_Horizontal, F.Cu at (383.4, 208.2)
- added D79: 1N4148, Diode_THT:D_DO-35_SOD27_P7.62mm_Horizontal, F.Cu at (402.9, 200.1)
- added D80: 1N4148, Diode_THT:D_DO-35_SOD27_P7.62mm_Horizontal, F.Cu at (363.8, 207.8)
- added D89: 1N4148, Diode_THT:D_DO-35_SOD27_P7.62mm_Horizontal, F.Cu at (550.4, 126.8)
- added D9: 1N4148, Diode_THT:D_DO-35_SOD27_P7.62mm_Horizontal, F.Cu at (373.6, 137.0)
- added D90: 1N4148, Diode_THT:D_DO-35_SOD27_P7.62mm_Horizontal, F.Cu at (595.2, 81.5)
- added D91: 1N4148, Diode_THT:D_DO-35_SOD27_P7.62mm_Horizontal, F.Cu at (540.6, 135.0)
- added D92: 1N4148, Diode_THT:D_DO-35_SOD27_P7.62mm_Horizontal, F.Cu at (576.1, 100.0)
- added D93: LED, LED_THT:LED_D3.0mm, F.Cu at (576.2, 113.7)
- added D94: LED, LED_THT:LED_D3.0mm, F.Cu at (595.8, 92.6)
- added D95: LED, LED_THT:LED_D3.0mm, F.Cu at (595.8, 88.1)
- added D96: LED, LED_THT:LED_D3.0mm, F.Cu at (576.2, 109.2)
- added D97: LED, LED_THT:LED_D3.0mm, F.Cu at (550.5, 135.5)
- added D98: LED, LED_THT:LED_D3.0mm, F.Cu at (586.0, 100.6)
- added D99: LED, LED_THT:LED_D3.0mm, F.Cu at (560.2, 127.8)
- added R1: 0, Resistor_THT:R_Axial_DIN0207_L6.3mm_D2.5mm_P7.62mm_Horizontal, F.Cu at (467.3, 70.0)
- added R10: 51, Resistor_THT:R_Axial_DIN0207_L6.3mm_D2.5mm_P7.62mm_Horizontal, F.Cu at (422.4, 130.1)
- added R100: 0, Resistor_THT:R_Axial_DIN0207_L6.3mm_D2.5mm_P7.62mm_Horizontal, F.Cu at (501.5, 127.1)
- added R101: 0, Resistor_THT:R_Axial_DIN0207_L6.3mm_D2.5mm_P7.62mm_Horizontal, F.Cu at (501.5, 130.1)
- added R102: 0, Resistor_THT:R_Axial_DIN0207_L6.3mm_D2.5mm_P7.62mm_Horizontal, F.Cu at (521.0, 132.7)
- added R11: 0, Resistor_THT:R_Axial_DIN0207_L6.3mm_D2.5mm_P7.62mm_Horizontal, F.Cu at (438.5, 115.0)
- added R12: 0, Resistor_THT:R_Axial_DIN0207_L6.3mm_D2.5mm_P7.62mm_Horizontal, F.Cu at (458.0, 91.7)
- added R13: 0, Resistor_THT:R_Axial_DIN0207_L6.3mm_D2.5mm_P7.62mm_Horizontal, F.Cu at (438.5, 105.8)
- added R14: 0, Resistor_THT:R_Axial_DIN0207_L6.3mm_D2.5mm_P7.62mm_Horizontal, F.Cu at (402.9, 132.2)
- added R15: 0, Resistor_THT:R_Axial_DIN0207_L6.3mm_D2.5mm_P7.62mm_Horizontal, F.Cu at (402.9, 135.2)
- added R16: 0, Resistor_THT:R_Axial_DIN0207_L6.3mm_D2.5mm_P7.62mm_Horizontal, F.Cu at (438.5, 99.8)
- added R17: 0, Resistor_THT:R_Axial_DIN0207_L6.3mm_D2.5mm_P7.62mm_Horizontal, F.Cu at (448.2, 97.7)
- added R18: 0, Resistor_THT:R_Axial_DIN0207_L6.3mm_D2.5mm_P7.62mm_Horizontal, F.Cu at (412.7, 132.7)
- added R19: 51, Resistor_THT:R_Axial_DIN0207_L6.3mm_D2.5mm_P7.62mm_Horizontal, F.Cu at (467.3, 79.2)
- added R2: 0, Resistor_THT:R_Axial_DIN0207_L6.3mm_D2.5mm_P7.62mm_Horizontal, F.Cu at (467.3, 73.1)
- added R20: 51, Resistor_THT:R_Axial_DIN0207_L6.3mm_D2.5mm_P7.62mm_Horizontal, F.Cu at (422.4, 127.1)
- added R21: 51, Resistor_THT:R_Axial_DIN0207_L6.3mm_D2.5mm_P7.62mm_Horizontal, F.Cu at (467.3, 82.2)
- added R22: 51, Resistor_THT:R_Axial_DIN0207_L6.3mm_D2.5mm_P7.62mm_Horizontal, F.Cu at (412.7, 135.7)
- added R23: 51, Resistor_THT:R_Axial_DIN0207_L6.3mm_D2.5mm_P7.62mm_Horizontal, F.Cu at (448.2, 100.8)
- added R24: 51, Resistor_THT:R_Axial_DIN0207_L6.3mm_D2.5mm_P7.62mm_Horizontal, F.Cu at (438.5, 108.9)
- added R25: 51, Resistor_THT:R_Axial_DIN0207_L6.3mm_D2.5mm_P7.62mm_Horizontal, F.Cu at (458.0, 88.7)
- added R26: 51, Resistor_THT:R_Axial_DIN0207_L6.3mm_D2.5mm_P7.62mm_Horizontal, F.Cu at (448.2, 103.8)
- added R27: 0, Resistor_THT:R_Axial_DIN0207_L6.3mm_D2.5mm_P7.62mm_Horizontal, F.Cu at (438.5, 102.8)
- added R28: 0, Resistor_THT:R_Axial_DIN0207_L6.3mm_D2.5mm_P7.62mm_Horizontal, F.Cu at (354.1, 127.1)
- added R29: 0, Resistor_THT:R_Axial_DIN0207_L6.3mm_D2.5mm_P7.62mm_Horizontal, F.Cu at (354.1, 130.1)
- added R3: 0, Resistor_THT:R_Axial_DIN0207_L6.3mm_D2.5mm_P7.62mm_Horizontal, F.Cu at (467.3, 76.1)
- added R30: 0, Resistor_THT:R_Axial_DIN0207_L6.3mm_D2.5mm_P7.62mm_Horizontal, F.Cu at (354.1, 133.2)
- added R31: 0, Resistor_THT:R_Axial_DIN0207_L6.3mm_D2.5mm_P7.62mm_Horizontal, F.Cu at (354.1, 136.2)
- added R32: 0, Resistor_THT:R_Axial_DIN0207_L6.3mm_D2.5mm_P7.62mm_Horizontal, F.Cu at (422.4, 133.2)
- added R33: 0, Resistor_THT:R_Axial_DIN0207_L6.3mm_D2.5mm_P7.62mm_Horizontal, F.Cu at (458.0, 94.8)
- added R34: 0, Resistor_THT:R_Axial_DIN0207_L6.3mm_D2.5mm_P7.62mm_Horizontal, F.Cu at (383.4, 132.2)
- added R35: 0, Resistor_THT:R_Axial_DIN0207_L6.3mm_D2.5mm_P7.62mm_Horizontal, F.Cu at (438.5, 167.9)
- added R36: 0, Resistor_THT:R_Axial_DIN0207_L6.3mm_D2.5mm_P7.62mm_Horizontal, F.Cu at (354.1, 200.3)
- added R37: 0, Resistor_THT:R_Axial_DIN0207_L6.3mm_D2.5mm_P7.62mm_Horizontal, F.Cu at (412.7, 200.3)
- added R38: 0, Resistor_THT:R_Axial_DIN0207_L6.3mm_D2.5mm_P7.62mm_Horizontal, F.Cu at (467.3, 152.4)
- added R39: 0, Resistor_THT:R_Axial_DIN0207_L6.3mm_D2.5mm_P7.62mm_Horizontal, F.Cu at (448.2, 171.0)
- added R4: 0, Resistor_THT:R_Axial_DIN0207_L6.3mm_D2.5mm_P7.62mm_Horizontal, F.Cu at (438.5, 112.0)
- added R40: 0, Resistor_THT:R_Axial_DIN0207_L6.3mm_D2.5mm_P7.62mm_Horizontal, F.Cu at (402.9, 208.0)
- added R41: 0, Resistor_THT:R_Axial_DIN0207_L6.3mm_D2.5mm_P7.62mm_Horizontal, F.Cu at (438.5, 180.1)
- added R42: 0, Resistor_THT:R_Axial_DIN0207_L6.3mm_D2.5mm_P7.62mm_Horizontal, F.Cu at (412.7, 203.4)
- added R43: 51, Resistor_THT:R_Axial_DIN0207_L6.3mm_D2.5mm_P7.62mm_Horizontal, F.Cu at (448.2, 167.9)
- added R44: 51, Resistor_THT:R_Axial_DIN0207_L6.3mm_D2.5mm_P7.62mm_Horizontal, F.Cu at (448.2, 164.9)
- added R45: 0, Resistor_THT:R_Axial_DIN0207_L6.3mm_D2.5mm_P7.62mm_Horizontal, F.Cu at (438.5, 171.0)
- added R46: 0, Resistor_THT:R_Axial_DIN0207_L6.3mm_D2.5mm_P7.62mm_Horizontal, F.Cu at (422.4, 200.3)
- added R47: 0, Resistor_THT:R_Axial_DIN0207_L6.3mm_D2.5mm_P7.62mm_Horizontal, F.Cu at (467.3, 143.3)
- added R48: 0, Resistor_THT:R_Axial_DIN0207_L6.3mm_D2.5mm_P7.62mm_Horizontal, F.Cu at (467.3, 146.3)
- added R49: 0, Resistor_THT:R_Axial_DIN0207_L6.3mm_D2.5mm_P7.62mm_Horizontal, F.Cu at (467.3, 149.4)
- added R5: 0, Resistor_THT:R_Axial_DIN0207_L6.3mm_D2.5mm_P7.62mm_Horizontal, F.Cu at (412.7, 129.6)
- added R50: 0, Resistor_THT:R_Axial_DIN0207_L6.3mm_D2.5mm_P7.62mm_Horizontal, F.Cu at (438.5, 174.0)
- added R51: 0, Resistor_THT:R_Axial_DIN0207_L6.3mm_D2.5mm_P7.62mm_Horizontal, F.Cu at (383.4, 200.3)
- added R52: 0, Resistor_THT:R_Axial_DIN0207_L6.3mm_D2.5mm_P7.62mm_Horizontal, F.Cu at (438.5, 189.3)
- added R53: 51, Resistor_THT:R_Axial_DIN0207_L6.3mm_D2.5mm_P7.62mm_Horizontal, F.Cu at (448.2, 180.1)
- added R54: 51, Resistor_THT:R_Axial_DIN0207_L6.3mm_D2.5mm_P7.62mm_Horizontal, F.Cu at (422.4, 203.4)
- added R55: 51, Resistor_THT:R_Axial_DIN0207_L6.3mm_D2.5mm_P7.62mm_Horizontal, F.Cu at (467.3, 158.5)
- added R56: 51, Resistor_THT:R_Axial_DIN0207_L6.3mm_D2.5mm_P7.62mm_Horizontal, F.Cu at (448.2, 177.1)
- added R57: 51, Resistor_THT:R_Axial_DIN0207_L6.3mm_D2.5mm_P7.62mm_Horizontal, F.Cu at (438.5, 186.2)
- added R58: 51, Resistor_THT:R_Axial_DIN0207_L6.3mm_D2.5mm_P7.62mm_Horizontal, F.Cu at (438.5, 177.1)
- added R59: 51, Resistor_THT:R_Axial_DIN0207_L6.3mm_D2.5mm_P7.62mm_Horizontal, F.Cu at (458.0, 165.0)
- added R6: 0, Resistor_THT:R_Axial_DIN0207_L6.3mm_D2.5mm_P7.62mm_Horizontal, F.Cu at (448.2, 91.6)
- added R60: 51, Resistor_THT:R_Axial_DIN0207_L6.3mm_D2.5mm_P7.62mm_Horizontal, F.Cu at (458.0, 161.9)
- added R61: 0, Resistor_THT:R_Axial_DIN0207_L6.3mm_D2.5mm_P7.62mm_Horizontal, F.Cu at (438.5, 183.2)
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- renumbered D9 to D41, D10 to D42, D11 to D43, D12 to D44, D13 to D45, D14 to D46, D15 to D47, D16 to D48, D17 to D81, D18 to D82, D19 to D83, D20 to D84, D21 to D85, D22 to D86, D23 to D87, D24 to D88, J3 to J2, J2 to J3, SW25 to SW1, SW6 to SW10, SW7 to SW11, SW8 to SW12, SW26 to SW2, SW9 to SW29, SW27 to SW3, SW10 to SW30, SW11 to SW31, SW12 to SW32, SW13 to SW33, SW14 to SW34, SW15 to SW35, SW16 to SW36, SW1 to SW5, SW17 to SW53, SW18 to SW54, SW19 to SW55, SW20 to SW56, SW21 to SW57, SW22 to SW58, SW23 to SW59, SW2 to SW6, SW24 to SW60, SW3 to SW7, SW4 to SW8, SW5 to SW9, U7 to U10, U2 to U3, U3 to U4, U4 to U6, U5 to U7, U6 to U9
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Connections:
- D41 pad 1: (no net) -> /sheet5C6557AC/GRID1
- D41 pad 2: (no net) -> Net-(D41-Pad2)
- D42 pad 1: (no net) -> /sheet5C6557AC/GRID2
- D42 pad 2: (no net) -> Net-(D41-Pad2)
- D43 pad 1: (no net) -> /sheet5C6557AC/GRID3
- D43 pad 2: (no net) -> Net-(D41-Pad2)
- D44 pad 1: (no net) -> /sheet5C6557AC/GRID4
- D44 pad 2: (no net) -> Net-(D41-Pad2)
- D45 pad 1: (no net) -> /sheet5C6557AC/GRID5
- D45 pad 2: (no net) -> Net-(D41-Pad2)
- D46 pad 1: (no net) -> /sheet5C6557AC/GRID6
- D46 pad 2: (no net) -> Net-(D41-Pad2)
- D47 pad 1: (no net) -> /sheet5C6557AC/GRID7
- D47 pad 2: (no net) -> Net-(D41-Pad2)
- D48 pad 1: (no net) -> /sheet5C6557AC/GRID8
- D48 pad 2: (no net) -> Net-(D41-Pad2)
- D5 pad 1: (no net) -> /TM1638 Module/GRID5
- D5 pad 2: (no net) -> Net-(D1-Pad2)
- D6 pad 1: (no net) -> /TM1638 Module/GRID6
- D6 pad 2: (no net) -> Net-(D1-Pad2)
- D7 pad 1: (no net) -> /TM1638 Module/GRID7
- D7 pad 2: (no net) -> Net-(D1-Pad2)
- D8 pad 1: (no net) -> /TM1638 Module/GRID8
- D8 pad 2: (no net) -> Net-(D1-Pad2)
- D81 pad 1: (no net) -> /sheet5C6559D3/GRID1
- D81 pad 2: (no net) -> Net-(D81-Pad2)
- D82 pad 1: (no net) -> /sheet5C6559D3/GRID2
- D82 pad 2: (no net) -> Net-(D81-Pad2)
- D83 pad 1: (no net) -> /sheet5C6559D3/GRID3
- D83 pad 2: (no net) -> Net-(D81-Pad2)
- D84 pad 1: (no net) -> /sheet5C6559D3/GRID4
- D84 pad 2: (no net) -> Net-(D81-Pad2)
- D85 pad 1: (no net) -> /sheet5C6559D3/GRID5
- D85 pad 2: (no net) -> Net-(D81-Pad2)
- D86 pad 1: (no net) -> /sheet5C6559D3/GRID6
- D86 pad 2: (no net) -> Net-(D81-Pad2)
- D87 pad 1: (no net) -> /sheet5C6559D3/GRID7
- D87 pad 2: (no net) -> Net-(D81-Pad2)
- D88 pad 1: (no net) -> /sheet5C6559D3/GRID8
- D88 pad 2: (no net) -> Net-(D81-Pad2)
- SW10 pad 1: (no net) -> /TM1638 Module/K1
- SW10 pad 2: (no net) -> /TM1638 Module/K1
- SW10 pad 3: (no net) -> Net-(D22-Pad1)
- SW10 pad 4: (no net) -> Net-(D22-Pad1)
- SW11 pad 1: (no net) -> /TM1638 Module/K1
- SW11 pad 2: (no net) -> /TM1638 Module/K1
- SW11 pad 3: (no net) -> Net-(D23-Pad1)
- SW11 pad 4: (no net) -> Net-(D23-Pad1)
- SW12 pad 1: (no net) -> /TM1638 Module/K1
- SW12 pad 2: (no net) -> /TM1638 Module/K1
- SW12 pad 3: (no net) -> Net-(D24-Pad1)
- SW12 pad 4: (no net) -> Net-(D24-Pad1)
- SW29 pad 1: (no net) -> /sheet5C6557AC/K1
- SW29 pad 2: (no net) -> /sheet5C6557AC/K1
- SW29 pad 3: (no net) -> Net-(D49-Pad1)
- SW29 pad 4: (no net) -> Net-(D49-Pad1)
- SW30 pad 1: (no net) -> /sheet5C6557AC/K1
- SW30 pad 2: (no net) -> /sheet5C6557AC/K1
- SW30 pad 3: (no net) -> Net-(D50-Pad1)
- SW30 pad 4: (no net) -> Net-(D50-Pad1)
- SW31 pad 1: (no net) -> /sheet5C6557AC/K1
- SW31 pad 2: (no net) -> /sheet5C6557AC/K1
- SW31 pad 3: (no net) -> Net-(D51-Pad1)
- SW31 pad 4: (no net) -> Net-(D51-Pad1)
- SW32 pad 1: (no net) -> /sheet5C6557AC/K1
- SW32 pad 2: (no net) -> /sheet5C6557AC/K1
- SW32 pad 3: (no net) -> Net-(D52-Pad1)
- SW32 pad 4: (no net) -> Net-(D52-Pad1)
- SW33 pad 1: (no net) -> /sheet5C6557AC/K1
- SW33 pad 2: (no net) -> /sheet5C6557AC/K1
- SW33 pad 3: (no net) -> Net-(D61-Pad1)
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
Commit message: board updated and schematic cleanup
Parts:
- added C10: 22pF, Capacitor_THT:C_Disc_D3.0mm_W2.0mm_P2.50mm, F.Cu at (212.4, 105.3)
- added C11: 100nF, Capacitor_THT:C_Disc_D3.0mm_W2.0mm_P2.50mm, F.Cu at (740.0, 90.2)
- added C12: 10uF, Capacitor_THT:CP_Radial_D6.3mm_P2.50mm, F.Cu at (734.3, 92.4)
- added C13: 100nF, Capacitor_THT:C_Disc_D3.0mm_W2.0mm_P2.50mm, F.Cu at (641.8, 126.5)
- added C14: 10uF, Capacitor_THT:CP_Radial_D6.3mm_P2.50mm, F.Cu at (636.0, 128.7)
- added C15: 100nF, Capacitor_THT:C_Disc_D3.0mm_W2.0mm_P2.50mm, F.Cu at (634.5, 120.6)
- added C16: 10uF, Capacitor_THT:CP_Radial_D6.3mm_P2.50mm, F.Cu at (655.9, 105.3)
- added C7: 10uF, Capacitor_THT:CP_Radial_D6.3mm_P2.50mm, F.Cu at (732.7, 77.6)
- added C8: 100nF, Capacitor_THT:C_Disc_D3.0mm_W2.0mm_P2.50mm, F.Cu at (731.5, 82.3)
- added C9: 22pF, Capacitor_THT:C_Disc_D3.0mm_W2.0mm_P2.50mm, F.Cu at (206.9, 105.4)
- added D121: 1N4148, Diode_THT:D_DO-35_SOD27_P7.62mm_Horizontal, F.Cu at (654.6, 88.4)
- added D122: 1N4148, Diode_THT:D_DO-35_SOD27_P7.62mm_Horizontal, F.Cu at (666.6, 78.9)
- added D123: 1N4148, Diode_THT:D_DO-35_SOD27_P7.62mm_Horizontal, F.Cu at (676.3, 75.9)
- added D124: 1N4148, Diode_THT:D_DO-35_SOD27_P7.62mm_Horizontal, F.Cu at (624.7, 120.6)
- added D125: 1N4148, Diode_THT:D_DO-35_SOD27_P7.62mm_Horizontal, F.Cu at (615.0, 120.6)
- added J5: USB_B, Connector_USB:USB_B_OST_USB-B1HSxx_Horizontal, F.Cu at (74.0, 89.7)
- added Q1: 2N7000, Package_TO_SOT_THT:TO-92_Inline, F.Cu at (721.6, 128.0)
- added Q2: 2N7000, Package_TO_SOT_THT:TO-92_Inline, F.Cu at (757.8, 71.3)
- added Q3: 2N7000, Package_TO_SOT_THT:TO-92_Inline, F.Cu at (723.7, 91.7)
- added Q4: 2N7000, Package_TO_SOT_THT:TO-92_Inline, F.Cu at (721.6, 140.3)
- added R103: 51, Resistor_THT:R_Axial_DIN0207_L6.3mm_D2.5mm_P7.62mm_Horizontal, F.Cu at (666.6, 76.1)
- added R104: 51, Resistor_THT:R_Axial_DIN0207_L6.3mm_D2.5mm_P7.62mm_Horizontal, F.Cu at (676.3, 73.1)
- added R105: 51, Resistor_THT:R_Axial_DIN0207_L6.3mm_D2.5mm_P7.62mm_Horizontal, F.Cu at (666.6, 73.1)
- added R106: 51, Resistor_THT:R_Axial_DIN0207_L6.3mm_D2.5mm_P7.62mm_Horizontal, F.Cu at (654.6, 91.2)
- added R107: 51, Resistor_THT:R_Axial_DIN0207_L6.3mm_D2.5mm_P7.62mm_Horizontal, F.Cu at (666.6, 70.0)
- added R108: 51, Resistor_THT:R_Axial_DIN0207_L6.3mm_D2.5mm_P7.62mm_Horizontal, F.Cu at (676.3, 70.0)
- added R109: 51, Resistor_THT:R_Axial_DIN0207_L6.3mm_D2.5mm_P7.62mm_Horizontal, F.Cu at (686.1, 73.1)
- added R110: 51, Resistor_THT:R_Axial_DIN0207_L6.3mm_D2.5mm_P7.62mm_Horizontal, F.Cu at (666.6, 84.8)
- added R111: 0, Resistor_THT:R_Axial_DIN0207_L6.3mm_D2.5mm_P7.62mm_Horizontal, F.Cu at (676.3, 81.7)
- added R112: 0, Resistor_THT:R_Axial_DIN0207_L6.3mm_D2.5mm_P7.62mm_Horizontal, F.Cu at (666.6, 81.7)
- added R113: 0, Resistor_THT:R_Axial_DIN0207_L6.3mm_D2.5mm_P7.62mm_Horizontal, F.Cu at (654.6, 100.4)
- added R114: 0, Resistor_THT:R_Axial_DIN0207_L6.3mm_D2.5mm_P7.62mm_Horizontal, F.Cu at (676.3, 78.7)
- added R115: 0, Resistor_THT:R_Axial_DIN0207_L6.3mm_D2.5mm_P7.62mm_Horizontal, F.Cu at (654.6, 97.3)
- added R116: 0, Resistor_THT:R_Axial_DIN0207_L6.3mm_D2.5mm_P7.62mm_Horizontal, F.Cu at (654.6, 94.3)
- added R117: 0, Resistor_THT:R_Axial_DIN0207_L6.3mm_D2.5mm_P7.62mm_Horizontal, F.Cu at (664.4, 88.7)
- added R118: 0, Resistor_THT:R_Axial_DIN0207_L6.3mm_D2.5mm_P7.62mm_Horizontal, F.Cu at (686.1, 70.0)
- added R119: 10k, Resistor_THT:R_Axial_DIN0207_L6.3mm_D2.5mm_P7.62mm_Horizontal, F.Cu at (711.4, 126.8)
- added R120: 10k, Resistor_THT:R_Axial_DIN0207_L6.3mm_D2.5mm_P7.62mm_Horizontal, F.Cu at (711.4, 129.8)
- added R121: 10k, Resistor_THT:R_Axial_DIN0207_L6.3mm_D2.5mm_P7.62mm_Horizontal, F.Cu at (747.6, 70.0)
- added R122: 10k, Resistor_THT:R_Axial_DIN0207_L6.3mm_D2.5mm_P7.62mm_Horizontal, F.Cu at (747.6, 73.1)
- added R123: 10k, Resistor_THT:R_Axial_DIN0207_L6.3mm_D2.5mm_P7.62mm_Horizontal, F.Cu at (713.6, 90.5)
- added R124: 10k, Resistor_THT:R_Axial_DIN0207_L6.3mm_D2.5mm_P7.62mm_Horizontal, F.Cu at (713.6, 93.5)
- added R125: 10k, Resistor_THT:R_Axial_DIN0207_L6.3mm_D2.5mm_P7.62mm_Horizontal, F.Cu at (711.4, 139.1)
- added R126: 10k, Resistor_THT:R_Axial_DIN0207_L6.3mm_D2.5mm_P7.62mm_Horizontal, F.Cu at (711.4, 142.1)
- added U11: CA56-12EWA, Display_7Segment:CA56-12EWA, F.Cu at (616.3, 144.3)
- added U12: TM1638, Package_SO:SOIC-28W_7.5x17.9mm_P1.27mm, F.Cu at (659.5, 77.8)
- added U13: CA56-12EWA, Display_7Segment:CA56-12EWA, F.Cu at (616.3, 87.6)
- added U14: CA56-12EWA, Display_7Segment:CA56-12EWA, F.Cu at (636.2, 87.6)
- added Y1: 20 MHz, Crystal:Crystal_HC49-U_Vertical, F.Cu at (211.8, 98.0)
- C1, C3: value 100nF -> 1nF; footprint Capacitor_SMD:C_0805_2012Metric -> Capacitor_THT:C_Disc_D3.0mm_W2.0mm_P2.50mm
- C2, C4, C6: value 10uF -> 100nF; footprint Capacitor_SMD:C_0805_2012Metric -> Capacitor_THT:C_Disc_D3.0mm_W2.0mm_P2.50mm
- C5: footprint Capacitor_SMD:C_0805_2012Metric -> Capacitor_THT:C_Disc_D3.0mm_W2.0mm_P2.50mm
- D1, D14, D15, D16, D17, D2, D3, D4, D41, D42, D43, D44, D45, D5, D54, D55, D56, D57, D81, D82, D83, D84, D85, D94, D95, D96, D97: value LED -> 1N4148; footprint LED_THT:LED_D3.0mm -> Diode_THT:D_DO-35_SOD27_P7.62mm_Horizontal
- D10, D101, D102, D103, D104, D105, D11, D12, D21, D22, D23, D24, D25, D49, D50, D51, D52, D61, D62, D63, D64, D65, D89, D9, D90, D91, D92: value 1N4148 -> LED; footprint Diode_THT:D_DO-35_SOD27_P7.62mm_Horizontal -> LED_THT:LED_D3.0mm
- J1: value USB_B -> footswitch; footprint Connector_USB:USB_B_OST_USB-B1HSxx_Horizontal -> beat707:trs
- J2: value AudioJack3_Ground -> click-out; footprint Connector_Audio:Jack_3.5mm_PJ311_Horizontal -> beat707:trs
- J3: value DIN-5_180degree -> MIDI-in; footprint beat707:DIN-Socket -> beat707:din-5
- J4: value DIN-5_180degree -> MIDI-out; footprint beat707:DIN-Socket -> beat707:din-5
- R1, R2, R5, R6, R8: value 0 -> 220
- R10: value 51 -> 10k
- R11, R12, R13, R14, R15, R16, R4, R7: value 0 -> 10k
- R19, R20, R21, R22, R23, R24, R43, R44, R53, R54, R55, R56, R57, R58, R77, R78, R87, R88, R89, R90, R91, R92: value 51 -> 0
- R3: value 0 -> 1k
- R35, R36, R37, R38, R39, R40, R41, R42, R69, R70, R71, R72, R73, R74, R75, R76: value 0 -> 51
- R9: value 51 -> 220
- SW1: value SW_Push -> Rotary_Encoder_Switch; footprint beat707:K2-1103SP-A4SW-04 -> Rotary_Encoder:RotaryEncoder_Alps_EC11E-Switch_Vertical_H20mm
- SW10, SW11, SW12, SW13, SW14, SW15, SW16, SW17, SW18, SW19, SW2, SW20, SW21, SW22, SW23, SW24, SW25, SW26, SW27, SW28, SW29, SW3, SW30, SW31, SW32, SW33, SW34, SW35, SW36, SW37, SW38, SW39, SW40, SW41, SW42, SW43, SW44, SW45, SW46, SW47, SW48, SW49, SW5, SW50, SW51, SW52, SW53, SW54, SW55, SW56, SW57, SW58, SW59, SW6, SW60, SW61, SW62, SW63, SW64, SW65, SW66, SW67, SW68, SW69, SW7, SW70, SW71, SW72, SW73, SW74, SW75, SW76, SW8, SW9: footprint beat707:K2-1103SP-A4SW-04 -> beat707:B3F-through-hole
- SW4: value Rotary_Encoder_Switch -> SW_Push; footprint Rotary_Encoder:RotaryEncoder_Alps_EC11E-Switch_Vertical_H20mm -> beat707:B3F-through-hole
- U1: value ATmega328-PU -> 6N138; footprint Package_DIP:DIP-28_W7.62mm -> Package_DIP:DIP-8_W7.62mm
- U2: value TM1638 -> 74HC14; footprint Package_SO:SOIC-28W_7.5x17.9mm_P1.27mm -> Package_DIP:DIP-14_W7.62mm
- U3: value CA56-12EWA -> MB85RS2MT; footprint Display_7Segment:CA56-12EWA -> Package_DIP:DIP-8_W7.62mm
- U4: value CA56-12EWA -> LP2950CZ-3.3G; footprint Display_7Segment:CA56-12EWA -> Package_TO_SOT_THT:TO-92_Inline
- U5: value TM1638 -> ATmega328-PU; footprint Package_SO:SOIC-28W_7.5x17.9mm_P1.27mm -> Package_DIP:DIP-28_W7.62mm
- U6, U9: value CA56-12EWA -> TM1638; footprint Display_7Segment:CA56-12EWA -> Package_SO:SOIC-28W_7.5x17.9mm_P1.27mm
- U8: value TM1638 -> CA56-12EWA; footprint Package_SO:SOIC-28W_7.5x17.9mm_P1.27mm -> Display_7Segment:CA56-12EWA
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Connections:
- C1 pad 1: +5V -> GND
- C1 pad 2: GND -> Net-(C1-Pad2)
- C2 pad 1: +5V -> GND
- C2 pad 2: GND -> Net-(C2-Pad2)
- C3 pad 1: +5V -> GND
- C3 pad 2: GND -> Net-(C3-Pad2)
- C5 pad 1: +5V -> GND
- C5 pad 2: GND -> +3V3
- D1 pad 1: /TM1638 Module/GRID1 -> Net-(D1-Pad1)
- D10 pad 1: Net-(D10-Pad1) -> /TM1638 Module/GRID5
- D10 pad 2: /TM1638 Module/SEG2 -> Net-(D10-Pad2)
- D100 pad 1: /sheet5C6559D3/GRID8 -> /sheet5C6559D3/GRID3
- D101 pad 1: Net-(D101-Pad1) -> /sheet5C6559D3/GRID4
- D101 pad 2: /sheet5C6559D3/SEG5 -> Net-(D100-Pad2)
- D102 pad 1: Net-(D102-Pad1) -> /sheet5C6559D3/GRID5
- D102 pad 2: /sheet5C6559D3/SEG6 -> Net-(D100-Pad2)
- D103 pad 1: Net-(D103-Pad1) -> /sheet5C6559D3/GRID6
- D103 pad 2: /sheet5C6559D3/SEG7 -> Net-(D100-Pad2)
- D104 pad 1: Net-(D104-Pad1) -> /sheet5C6559D3/GRID7
- D104 pad 2: /sheet5C6559D3/SEG8 -> Net-(D100-Pad2)
- D105 pad 1: Net-(D105-Pad1) -> /sheet5C6559D3/GRID8
- D105 pad 2: /sheet5C6559D3/SEG1 -> Net-(D100-Pad2)
- D106 pad 2: /sheet5C6559D3/SEG2 -> /sheet5C6559D3/SEG5
- D107 pad 2: /sheet5C6559D3/SEG3 -> /sheet5C6559D3/SEG6
- D108 pad 2: /sheet5C6559D3/SEG4 -> /sheet5C6559D3/SEG7
- D109 pad 2: /sheet5C6559D3/SEG5 -> /sheet5C6559D3/SEG8
- D11 pad 1: Net-(D11-Pad1) -> /TM1638 Module/GRID6
- D11 pad 2: /TM1638 Module/SEG3 -> Net-(D10-Pad2)
- D110 pad 2: /sheet5C6559D3/SEG6 -> /sheet5C6559D3/SEG1
- D111 pad 2: /sheet5C6559D3/SEG7 -> /sheet5C6559D3/SEG2
- D112 pad 2: /sheet5C6559D3/SEG8 -> /sheet5C6559D3/SEG3
- D113 pad 2: /sheet5C6559D3/SEG1 -> /sheet5C6559D3/SEG4
- D114 pad 2: /sheet5C6559D3/SEG2 -> /sheet5C6559D3/SEG5
- D115 pad 2: /sheet5C6559D3/SEG3 -> /sheet5C6559D3/SEG6
- D116 pad 2: /sheet5C6559D3/SEG4 -> /sheet5C6559D3/SEG7
- D117 pad 2: /sheet5C6559D3/SEG5 -> /sheet5C6559D3/SEG8
- D118 pad 2: /sheet5C6559D3/SEG6 -> /sheet5C6559D3/SEG1
- D119 pad 2: /sheet5C6559D3/SEG7 -> /sheet5C6559D3/SEG2
- D12 pad 1: Net-(D12-Pad1) -> /TM1638 Module/GRID7
- D12 pad 2: /TM1638 Module/SEG4 -> Net-(D10-Pad2)
- D120 pad 2: /sheet5C6559D3/SEG8 -> /sheet5C6559D3/SEG3
- D13 pad 1: /TM1638 Module/GRID1 -> /TM1638 Module/GRID8
- D13 pad 2: Net-(D13-Pad2) -> Net-(D10-Pad2)
- D14 pad 1: /TM1638 Module/GRID2 -> Net-(D14-Pad1)
- D14 pad 2: Net-(D13-Pad2) -> /TM1638 Module/SEG1
- D15 pad 1: /TM1638 Module/GRID3 -> Net-(D15-Pad1)
- D15 pad 2: Net-(D13-Pad2) -> /TM1638 Module/SEG2
- D16 pad 1: /TM1638 Module/GRID4 -> Net-(D16-Pad1)
- D16 pad 2: Net-(D13-Pad2) -> /TM1638 Module/SEG3
- D17 pad 1: /TM1638 Module/GRID5 -> Net-(D17-Pad1)
- D17 pad 2: Net-(D13-Pad2) -> /TM1638 Module/SEG4
- D18 pad 1: /TM1638 Module/GRID6 -> /TM1638 Module/GRID1
- D18 pad 2: Net-(D13-Pad2) -> Net-(D18-Pad2)
- D19 pad 1: /TM1638 Module/GRID7 -> /TM1638 Module/GRID2
- D19 pad 2: Net-(D13-Pad2) -> Net-(D18-Pad2)
- D2 pad 1: /TM1638 Module/GRID2 -> +5V
- D2 pad 2: Net-(D1-Pad2) -> Net-(C1-Pad2)
- D20 pad 1: /TM1638 Module/GRID8 -> /TM1638 Module/GRID3
- D20 pad 2: Net-(D13-Pad2) -> Net-(D18-Pad2)
- D21 pad 1: Net-(D21-Pad1) -> /TM1638 Module/GRID4
- D21 pad 2: /TM1638 Module/SEG5 -> Net-(D18-Pad2)
- D22 pad 1: Net-(D22-Pad1) -> /TM1638 Module/GRID5
- D22 pad 2: /TM1638 Module/SEG6 -> Net-(D18-Pad2)
- D23 pad 1: Net-(D23-Pad1) -> /TM1638 Module/GRID6
- D23 pad 2: /TM1638 Module/SEG7 -> Net-(D18-Pad2)
- D24 pad 1: Net-(D24-Pad1) -> /TM1638 Module/GRID7
- D24 pad 2: /TM1638 Module/SEG8 -> Net-(D18-Pad2)
- D25 pad 1: Net-(D25-Pad1) -> /TM1638 Module/GRID8
- D25 pad 2: /TM1638 Module/SEG1 -> Net-(D18-Pad2)
- D26 pad 2: /TM1638 Module/SEG2 -> /TM1638 Module/SEG5
- D27 pad 2: /TM1638 Module/SEG3 -> /TM1638 Module/SEG6
- D28 pad 2: /TM1638 Module/SEG4 -> /TM1638 Module/SEG7
- D29 pad 2: /TM1638 Module/SEG5 -> /TM1638 Module/SEG8
- D3 pad 1: /TM1638 Module/GRID3 -> Net-(C1-Pad2)
- D3 pad 2: Net-(D1-Pad2) -> GND
- D30 pad 2: /TM1638 Module/SEG6 -> /TM1638 Module/SEG1
- D31 pad 2: /TM1638 Module/SEG7 -> /TM1638 Module/SEG2
- D32 pad 2: /TM1638 Module/SEG8 -> /TM1638 Module/SEG3
- D33 pad 2: /TM1638 Module/SEG1 -> /TM1638 Module/SEG4
- D34 pad 2: /TM1638 Module/SEG2 -> /TM1638 Module/SEG5
- D35 pad 2: /TM1638 Module/SEG3 -> /TM1638 Module/SEG6
- D36 pad 2: /TM1638 Module/SEG4 -> /TM1638 Module/SEG7
- D37 pad 2: /TM1638 Module/SEG5 -> /TM1638 Module/SEG8
- D38 pad 2: /TM1638 Module/SEG6 -> /TM1638 Module/SEG1
- D39 pad 2: /TM1638 Module/SEG7 -> /TM1638 Module/SEG2
- D4 pad 1: /TM1638 Module/GRID4 -> +5V
- D4 pad 2: Net-(D1-Pad2) -> Net-(C3-Pad2)
- D40 pad 2: /TM1638 Module/SEG8 -> /TM1638 Module/SEG3
- D41 pad 1: /sheet5C6557AC/GRID1 -> Net-(D41-Pad1)
- D41 pad 2: Net-(D41-Pad2) -> /TM1638 Module/SEG4
- D42 pad 1: /sheet5C6557AC/GRID2 -> Net-(D42-Pad1)
- D42 pad 2: Net-(D41-Pad2) -> /TM1638 Module/SEG5
- D43 pad 1: /sheet5C6557AC/GRID3 -> Net-(D43-Pad1)
- D43 pad 2: Net-(D41-Pad2) -> /TM1638 Module/SEG6
- D44 pad 1: /sheet5C6557AC/GRID4 -> Net-(D44-Pad1)
- D44 pad 2: Net-(D41-Pad2) -> /TM1638 Module/SEG7
- D45 pad 1: /sheet5C6557AC/GRID5 -> Net-(D45-Pad1)
- D45 pad 2: Net-(D41-Pad2) -> /TM1638 Module/SEG8
- D46 pad 1: /sheet5C6557AC/GRID6 -> /sheet5C6557AC/GRID1
- D46 pad 2: Net-(D41-Pad2) -> Net-(D46-Pad2)
- D47 pad 1: /sheet5C6557AC/GRID7 -> /sheet5C6557AC/GRID2
- D47 pad 2: Net-(D41-Pad2) -> Net-(D46-Pad2)
- D48 pad 1: /sheet5C6557AC/GRID8 -> /sheet5C6557AC/GRID3
- D48 pad 2: Net-(D41-Pad2) -> Net-(D46-Pad2)
- D49 pad 1: Net-(D49-Pad1) -> /sheet5C6557AC/GRID4
- D49 pad 2: /sheet5C6557AC/SEG1 -> Net-(D46-Pad2)
- D5 pad 1: /TM1638 Module/GRID5 -> Net-(C3-Pad2)
- D5 pad 2: Net-(D1-Pad2) -> GND
- D50 pad 1: Net-(D50-Pad1) -> /sheet5C6557AC/GRID5
- D50 pad 2: /sheet5C6557AC/SEG2 -> Net-(D46-Pad2)
- D51 pad 1: Net-(D51-Pad1) -> /sheet5C6557AC/GRID6
- D51 pad 2: /sheet5C6557AC/SEG3 -> Net-(D46-Pad2)
- D52 pad 1: Net-(D52-Pad1) -> /sheet5C6557AC/GRID7
- D52 pad 2: /sheet5C6557AC/SEG4 -> Net-(D46-Pad2)
- D53 pad 1: /sheet5C6557AC/GRID1 -> /sheet5C6557AC/GRID8
- D53 pad 2: Net-(D53-Pad2) -> Net-(D46-Pad2)
- D54 pad 1: /sheet5C6557AC/GRID2 -> Net-(D54-Pad1)
- D54 pad 2: Net-(D53-Pad2) -> /sheet5C6557AC/SEG1
- D55 pad 1: /sheet5C6557AC/GRID3 -> Net-(D55-Pad1)
- D55 pad 2: Net-(D53-Pad2) -> /sheet5C6557AC/SEG2
- D56 pad 1: /sheet5C6557AC/GRID4 -> Net-(D56-Pad1)
- D56 pad 2: Net-(D53-Pad2) -> /sheet5C6557AC/SEG3
- D57 pad 1: /sheet5C6557AC/GRID5 -> Net-(D57-Pad1)
- D57 pad 2: Net-(D53-Pad2) -> /sheet5C6557AC/SEG4
- D58 pad 1: /sheet5C6557AC/GRID6 -> /sheet5C6557AC/GRID1
- D58 pad 2: Net-(D53-Pad2) -> Net-(D58-Pad2)
- D59 pad 1: /sheet5C6557AC/GRID7 -> /sheet5C6557AC/GRID2
- D59 pad 2: Net-(D53-Pad2) -> Net-(D58-Pad2)
- D6 pad 1: /TM1638 Module/GRID6 -> /TM1638 Module/GRID1
- D6 pad 2: Net-(D1-Pad2) -> Net-(D10-Pad2)
- D60 pad 1: /sheet5C6557AC/GRID8 -> /sheet5C6557AC/GRID3
- D60 pad 2: Net-(D53-Pad2) -> Net-(D58-Pad2)
- D61 pad 1: Net-(D61-Pad1) -> /sheet5C6557AC/GRID4
- D61 pad 2: /sheet5C6557AC/SEG5 -> Net-(D58-Pad2)
- D62 pad 1: Net-(D62-Pad1) -> /sheet5C6557AC/GRID5
- D62 pad 2: /sheet5C6557AC/SEG6 -> Net-(D58-Pad2)
- D63 pad 1: Net-(D63-Pad1) -> /sheet5C6557AC/GRID6
- D63 pad 2: /sheet5C6557AC/SEG7 -> Net-(D58-Pad2)
- D64 pad 1: Net-(D64-Pad1) -> /sheet5C6557AC/GRID7
- D64 pad 2: /sheet5C6557AC/SEG8 -> Net-(D58-Pad2)
- D65 pad 1: Net-(D65-Pad1) -> /sheet5C6557AC/GRID8
- D65 pad 2: /sheet5C6557AC/SEG1 -> Net-(D58-Pad2)
- D66 pad 2: /sheet5C6557AC/SEG2 -> /sheet5C6557AC/SEG5
- D67 pad 2: /sheet5C6557AC/SEG3 -> /sheet5C6557AC/SEG6
- D68 pad 2: /sheet5C6557AC/SEG4 -> /sheet5C6557AC/SEG7
- D69 pad 2: /sheet5C6557AC/SEG5 -> /sheet5C6557AC/SEG8
- D7 pad 1: /TM1638 Module/GRID7 -> /TM1638 Module/GRID2
- D7 pad 2: Net-(D1-Pad2) -> Net-(D10-Pad2)
- D70 pad 2: /sheet5C6557AC/SEG6 -> /sheet5C6557AC/SEG1
- D71 pad 2: /sheet5C6557AC/SEG7 -> /sheet5C6557AC/SEG2
- D72 pad 2: /sheet5C6557AC/SEG8 -> /sheet5C6557AC/SEG3
- D73 pad 2: /sheet5C6557AC/SEG1 -> /sheet5C6557AC/SEG4
- D74 pad 2: /sheet5C6557AC/SEG2 -> /sheet5C6557AC/SEG5
- D75 pad 2: /sheet5C6557AC/SEG3 -> /sheet5C6557AC/SEG6
- D76 pad 2: /sheet5C6557AC/SEG4 -> /sheet5C6557AC/SEG7
- D77 pad 2: /sheet5C6557AC/SEG5 -> /sheet5C6557AC/SEG8
- D78 pad 2: /sheet5C6557AC/SEG6 -> /sheet5C6557AC/SEG1
- D79 pad 2: /sheet5C6557AC/SEG7 -> /sheet5C6557AC/SEG2
- D8 pad 1: /TM1638 Module/GRID8 -> /TM1638 Module/GRID3
- D8 pad 2: Net-(D1-Pad2) -> Net-(D10-Pad2)
- D80 pad 2: /sheet5C6557AC/SEG8 -> /sheet5C6557AC/SEG3
- D81 pad 1: /sheet5C6559D3/GRID1 -> Net-(D81-Pad1)
- D81 pad 2: Net-(D81-Pad2) -> /sheet5C6557AC/SEG4
- D82 pad 1: /sheet5C6559D3/GRID2 -> Net-(D82-Pad1)
- D82 pad 2: Net-(D81-Pad2) -> /sheet5C6557AC/SEG5
- D83 pad 1: /sheet5C6559D3/GRID3 -> Net-(D83-Pad1)
- D83 pad 2: Net-(D81-Pad2) -> /sheet5C6557AC/SEG6
- D84 pad 1: /sheet5C6559D3/GRID4 -> Net-(D84-Pad1)
- D84 pad 2: Net-(D81-Pad2) -> /sheet5C6557AC/SEG7
- D85 pad 1: /sheet5C6559D3/GRID5 -> Net-(D85-Pad1)
- D85 pad 2: Net-(D81-Pad2) -> /sheet5C6557AC/SEG8
- D86 pad 1: /sheet5C6559D3/GRID6 -> /sheet5C6559D3/GRID1
- D86 pad 2: Net-(D81-Pad2) -> Net-(D86-Pad2)
- D87 pad 1: /sheet5C6559D3/GRID7 -> /sheet5C6559D3/GRID2
- D87 pad 2: Net-(D81-Pad2) -> Net-(D86-Pad2)
- D88 pad 1: /sheet5C6559D3/GRID8 -> /sheet5C6559D3/GRID3
- D88 pad 2: Net-(D81-Pad2) -> Net-(D86-Pad2)
- D89 pad 1: Net-(D89-Pad1) -> /sheet5C6559D3/GRID4
- D89 pad 2: /sheet5C6559D3/SEG1 -> Net-(D86-Pad2)
- D9 pad 1: Net-(D9-Pad1) -> /TM1638 Module/GRID4
- D9 pad 2: /TM1638 Module/SEG1 -> Net-(D10-Pad2)
- D90 pad 1: Net-(D90-Pad1) -> /sheet5C6559D3/GRID5
- D90 pad 2: /sheet5C6559D3/SEG2 -> Net-(D86-Pad2)
- D91 pad 1: Net-(D91-Pad1) -> /sheet5C6559D3/GRID6
- D91 pad 2: /sheet5C6559D3/SEG3 -> Net-(D86-Pad2)
- D92 pad 1: Net-(D92-Pad1) -> /sheet5C6559D3/GRID7
- D92 pad 2: /sheet5C6559D3/SEG4 -> Net-(D86-Pad2)
- D93 pad 1: /sheet5C6559D3/GRID1 -> /sheet5C6559D3/GRID8
- D93 pad 2: Net-(D100-Pad2) -> Net-(D86-Pad2)
- D94 pad 1: /sheet5C6559D3/GRID2 -> Net-(D94-Pad1)
- D94 pad 2: Net-(D100-Pad2) -> /sheet5C6559D3/SEG1
- D95 pad 1: /sheet5C6559D3/GRID3 -> Net-(D95-Pad1)
- D95 pad 2: Net-(D100-Pad2) -> /sheet5C6559D3/SEG2
- D96 pad 1: /sheet5C6559D3/GRID4 -> Net-(D96-Pad1)
- D96 pad 2: Net-(D100-Pad2) -> /sheet5C6559D3/SEG3
- D97 pad 1: /sheet5C6559D3/GRID5 -> Net-(D97-Pad1)
- D97 pad 2: Net-(D100-Pad2) -> /sheet5C6559D3/SEG4
- D98 pad 1: /sheet5C6559D3/GRID6 -> /sheet5C6559D3/GRID1
- D99 pad 1: /sheet5C6559D3/GRID7 -> /sheet5C6559D3/GRID2
- J1 pad 5: Net-(J1-Pad5) -> (no net)
- J3 pad 4: (no net) -> Net-(J3-Pad4)
- J3 pad 5: (no net) -> Net-(D1-Pad2)
- J4 pad 2: (no net) -> GND
- J4 pad 4: (no net) -> Net-(J4-Pad4)
- J4 pad 5: (no net) -> Net-(C3-Pad2)
- R1 pad 1: Net-(D9-Pad1) -> Net-(J4-Pad4)
- R1 pad 2: /TM1638 Module/K1 -> +5V
- R10 pad 1: Net-(R10-Pad1) -> +5V
- R10 pad 2: Net-(D1-Pad2) -> Net-(R10-Pad2)
- R100 pad 1: Net-(D118-Pad1) -> Net-(D115-Pad1)
- R100 pad 2: /sheet5C6559D3/K3 -> /sheet5C6559D3/K2
- R101 pad 1: Net-(D119-Pad1) -> Net-(D116-Pad1)
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