File: kicad/beat707/beat707.kicad_pcb (KiCad board)
At the start: 2 copper layers, 292.1 x 134.6 mm, 367 parts, among them J1 footswitch, J2 click-out, J3 MIDI-in, J4 MIDI-out, J5 USB_B, Q1 2N7000, Q2 2N7000, Q3 2N7000, Q4 2N7000, SW1 Rotary_Encoder_Switch, SW10 SW_Push, SW11 SW_Push, SW12 SW_Push, SW13 SW_Push, SW14 SW_Push, SW15 SW_Push, SW16 SW_Push, SW17 SW_Push, SW18 SW_Push, SW19 SW_Push, SW2 SW_Push, SW20 SW_Push, SW21 SW_Push, SW22 SW_Push, SW23 SW_Push, SW24 SW_Push, SW25 SW_Push, SW26 SW_Push, SW27 SW_Push, SW28 SW_Push, SW29 SW_Push, SW3 SW_Push, SW30 SW_Push, SW31 SW_Push, SW32 SW_Push, SW33 SW_Push, SW34 SW_Push, SW35 SW_Push, SW36 SW_Push, SW37 SW_Push, SW38 SW_Push, SW39 SW_Push, SW4 SW_Push, SW40 SW_Push, SW41 SW_Push, SW42 SW_Push, SW43 SW_Push, SW44 SW_Push, SW45 SW_Push, SW46 SW_Push, SW47 SW_Push, SW48 SW_Push, SW49 SW_Push, SW5 SW_Push, SW50 SW_Push, SW51 SW_Push, SW52 SW_Push, SW53 SW_Push, SW54 SW_Push, SW55 SW_Push, SW56 SW_Push, SW57 SW_Push, SW58 SW_Push, SW59 SW_Push, SW6 SW_Push, SW60 SW_Push, SW61 SW_Push, SW62 SW_Push, SW63 SW_Push, SW64 SW_Push, SW65 SW_Push, SW66 SW_Push, SW67 SW_Push, SW68 SW_Push, SW69 SW_Push, SW7 SW_Push, SW70 SW_Push, SW71 SW_Push, SW72 SW_Push, SW73 SW_Push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

Commit message: components on pcb sorted, not needed = below
Parts:
- moved C11 645.2 mm to (95.2, 115.6)
- moved C12 639.7 mm to (95.2, 123.2)
- moved R121 572.0 mm to (177.8, 120.7)
- moved C13 539.0 mm to (102.9, 115.6)
- moved C14 533.2 mm to (102.9, 123.2)
- moved Q4 529.4 mm to (193.0, 110.5)
- moved R122 523.1 mm to (226.1, 113.0)
- moved Q1 522.5 mm to (199.4, 110.5)
- moved C7 497.0 mm to (236.3, 101.6)
- moved C8 494.8 mm to (237.4, 110.2)
- moved R76 461.8 mm to (133.5, 96.4), turned to 180 degrees
- moved R69 453.7 mm to (133.5, 123.0), turned to 180 degrees
- moved R71 453.0 mm to (133.5, 115.4), turned to 180 degrees
- moved R74 442.6 mm to (133.5, 104.0), turned to 180 degrees
- moved R75 442.6 mm to (133.5, 100.2), turned to 180 degrees
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
Commit message: making brainboard space
mute leds moved to 4x4 block upper right (will change leds to come from right side tm1638 for easier routing), added spaces between 4 steps, TM1638 part placement = just a try, brainboard parts not placed at all, just dragged for checking space
Parts:
- moved D46 181.2 mm to (252.7, 74.9)
- moved D47 175.5 mm to (261.6, 74.9)
- moved R119 172.3 mm to (167.6, 138.4)
- moved R120 172.3 mm to (167.6, 132.1)
- moved R12 172.3 mm to (141.0, 135.9)
- moved R126 172.3 mm to (163.8, 143.5)
- moved R3 172.3 mm to (141.0, 129.5)
- moved R6 172.3 mm to (141.0, 142.2)
- moved R123 172.3 mm to (154.9, 133.3)
- moved R124 172.3 mm to (154.9, 128.3)
- moved D48 172.1 mm to (270.5, 74.9)
- moved D49 168.7 mm to (279.4, 74.9)
- moved R125 154.4 mm to (179.1, 128.3)
- moved R5 151.8 mm to (176.5, 96.5)
- moved R4 131.6 mm to (175.3, 105.4)
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Other:
- board size 292.1 x 134.6 mm -> 273.1 x 134.6 mm
- board text added: "PLAY/REC"
- board text removed: "PLAY RECORD"

Commit message: Update beat707.kicad_pcb
semi final UI element placement & board size. missing: optional mounting holes (square footprint)
Parts:
- moved D58 221.5 mm to (299.1, 116.8)
- moved D59 216.1 mm to (306.1, 116.8)
- moved D60 210.6 mm to (313.1, 116.8)
- moved D61 205.2 mm to (320.0, 116.8)
- moved D86 196.9 mm to (88.9, 201.9)
- moved D87 193.7 mm to (101.6, 201.9)
- moved D88 190.6 mm to (114.3, 201.9)
- moved D89 187.5 mm to (127.0, 201.9)
- moved D62 168.8 mm to (299.1, 123.8)
- moved D63 163.4 mm to (306.1, 123.8)
- moved D64 158.1 mm to (313.1, 123.8)
- moved D65 152.8 mm to (320.0, 123.8)
- moved D90 149.2 mm to (142.2, 201.9)
- moved D91 146.4 mm to (154.9, 201.9)
- moved D92 143.7 mm to (167.6, 201.9)
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Other:
- board size 273.1 x 134.6 mm -> 279.4 x 134.6 mm
- board text added: "CONNECTOR SPACING UNOPTIMIZED GERT: CHECK WITH REAL LIFE CABLES"
- board text added: "INDEX FINGER SPACE (UNOPTIMIZED)"
- board text added: "OPTIONAL SILKSCREEN LINE"
- board text added: "OPTIONAL SILKSCREEN LINE 1"
- board text added: "PLEASE MIND TO PLACE ELECTROLYTE CAPS SAFE: AWAY FROM USER INTERFACE - NOT ON THE EDGE"
- board text added: "THUMB REST SPACE (UNOPTIMIZED)"
- board text added: "TRACK ACTIVITY"

Commit message: Update beat707.kicad_pcb
first try for step silkscreen
Parts:
- moved C3 12.8 mm to (173.4, 173.4)
- moved C4 12.8 mm to (216.5, 151.8)
- moved C5 12.8 mm to (184.8, 139.1)
- moved D1 12.8 mm to (163.2, 151.8)
- moved D2 12.8 mm to (191.1, 163.2)
- moved D4 12.8 mm to (191.1, 169.5)
- moved R1 12.8 mm to (205.1, 160.7)
- moved R124 12.8 mm to (151.8, 156.8)
- moved R9 12.8 mm to (205.1, 167.0)
- moved D5 12.8 mm to (163.2, 148.0)
- moved R123 12.8 mm to (151.8, 161.9)
- moved R13 12.8 mm to (205.1, 172.1)
- moved R2 12.8 mm to (205.1, 154.3)
- moved R5 12.8 mm to (173.4, 125.1)
- moved C10 12.8 mm to (213.0, 145.3)
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Other:
- board size 279.4 x 134.6 mm -> 274.3 x 134.6 mm
- board text added: "1"
- board text added: "10"
- board text added: "11"
- board text added: "12"
- board text added: "13"
- board text added: "14"
- board text added: "15"
- board text added: "16"
- board text added: "2"
- board text added: "3"
- board text added: "4"
- board text added: "5"
- board text added: "6."
- board text added: "7"
- board text added: "8"
- board text added: "9."
- board text removed: "OPTIONAL SILKSCREEN LINE 1"

Commit message: restored deleted files and added all 3D models
Parts:
- removed Q2, Q3, Q4: 2N7000, Package_TO_SOT_THT:TO-92_Inline
- added J6: free IO, Connector_PinHeader_2.54mm:PinHeader_1x01_P2.54mm_Vertical, F.Cu at (390.3, 92.5)
- C1, C3: footprint Capacitor_THT:C_Disc_D3.0mm_W2.0mm_P2.50mm -> Capacitor_THT:C_Disc_D8.0mm_W5.0mm_P7.50mm
- R119, R121, R124: value 10k -> 2.2k
- R120, R122, R123, R125, R126: value 10k -> 3.3k
- moved R123 238.9 mm to (379.7, 90.4)
- moved R126 231.7 mm to (379.7, 96.5)
- moved R124 226.4 mm to (370.0, 96.5)
- moved R119 220.4 mm to (370.0, 87.4)
- moved R120 217.2 mm to (370.0, 90.4)
- moved R121 214.2 mm to (379.7, 87.4)
- moved R125 213.5 mm to (379.7, 93.5)
- moved Q1 200.2 mm to (389.9, 88.6)
- moved R122 157.2 mm to (370.0, 93.5)
- moved R13 79.5 mm to (129.5, 147.3)
- moved C3 78.6 mm to (227.3, 116.2)
- moved R1 77.8 mm to (129.5, 142.2)
- moved U1 77.0 mm to (210.8, 116.8), turned to 270 degrees
- moved D5 76.1 mm to (234.9, 122.6), turned to 180 degrees
- moved D1 59.9 mm to (208.9, 113.0), turned to 180 degrees
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Connections:
- Q1 pad 1: /Sheet5CCE7B2F/low-side -> Net-(Q1-Pad1)
- Q1 pad 3: FRAM-SCK -> FRAM-SO
- R119 pad 1: /Sheet5CCE7B2F/low-side -> Net-(R119-Pad1)
- R119 pad 2: +3V3 -> FRAM-~CS
- R120 pad 1: FRAM-SCK -> GND
- R120 pad 2: +5V -> Net-(R119-Pad1)
- R121 pad 1: /sheet5CD0BEEF/low-side -> Net-(R121-Pad1)
- R121 pad 2: +3V3 -> FRAM-SI
- R122 pad 1: FRAM-SI -> GND
- R122 pad 2: +5V -> Net-(R121-Pad1)
- R123 pad 1: /sheet5CD14929/low-side -> Net-(Q1-Pad1)
- R124 pad 1: FRAM-SO -> Net-(R124-Pad1)
- R124 pad 2: +5V -> FRAM-SCK
- R125 pad 1: /sheet5CD1D363/low-side -> GND
- R125 pad 2: +3V3 -> Net-(R124-Pad1)
- R126 pad 1: FRAM-~CS -> FRAM-SO
- SW10 pad 1: /TM1638 Module/K1 -> (no net)
- SW10 pad 2: /TM1638 Module/K1 -> (no net)
- SW10 pad 3: Net-(D27-Pad1) -> (no net)
- SW11 pad 1: /TM1638 Module/K1 -> (no net)
- SW11 pad 2: /TM1638 Module/K1 -> (no net)
- SW11 pad 3: Net-(D28-Pad1) -> (no net)
- SW12 pad 1: /TM1638 Module/K1 -> (no net)
- SW12 pad 2: /TM1638 Module/K1 -> (no net)
- SW12 pad 3: Net-(D29-Pad1) -> (no net)
- SW13 pad 1: /TM1638 Module/K2 -> (no net)
- SW13 pad 2: /TM1638 Module/K2 -> (no net)
- SW13 pad 3: Net-(D30-Pad1) -> (no net)
- SW14 pad 1: /TM1638 Module/K2 -> (no net)
- SW14 pad 2: /TM1638 Module/K2 -> (no net)
- SW14 pad 3: Net-(D31-Pad1) -> (no net)
- SW15 pad 1: /TM1638 Module/K2 -> (no net)
- SW15 pad 2: /TM1638 Module/K2 -> (no net)
- SW15 pad 3: Net-(D32-Pad1) -> (no net)
- SW16 pad 1: /TM1638 Module/K2 -> (no net)
- SW16 pad 2: /TM1638 Module/K2 -> (no net)
- SW16 pad 3: Net-(D33-Pad1) -> (no net)
- SW17 pad 1: /TM1638 Module/K2 -> (no net)
- SW17 pad 2: /TM1638 Module/K2 -> (no net)
- SW17 pad 3: Net-(D34-Pad1) -> (no net)
- SW18 pad 1: /TM1638 Module/K2 -> (no net)
- SW18 pad 2: /TM1638 Module/K2 -> (no net)
- SW18 pad 3: Net-(D35-Pad1) -> (no net)
- SW19 pad 1: /TM1638 Module/K2 -> (no net)
- SW19 pad 2: /TM1638 Module/K2 -> (no net)
- SW19 pad 3: Net-(D36-Pad1) -> (no net)
- SW20 pad 1: /TM1638 Module/K2 -> (no net)
- SW20 pad 2: /TM1638 Module/K2 -> (no net)
- SW20 pad 3: Net-(D37-Pad1) -> (no net)
- SW21 pad 1: /TM1638 Module/K3 -> (no net)
- SW21 pad 2: /TM1638 Module/K3 -> (no net)
- SW21 pad 3: Net-(D38-Pad1) -> (no net)
- SW22 pad 1: /TM1638 Module/K3 -> (no net)
- SW22 pad 2: /TM1638 Module/K3 -> (no net)
- SW22 pad 3: Net-(D39-Pad1) -> (no net)
- SW23 pad 1: /TM1638 Module/K3 -> (no net)
- SW23 pad 2: /TM1638 Module/K3 -> (no net)
- SW23 pad 3: Net-(D40-Pad1) -> (no net)
- SW24 pad 1: /TM1638 Module/K3 -> (no net)
- SW24 pad 2: /TM1638 Module/K3 -> (no net)
- SW24 pad 3: Net-(D41-Pad1) -> (no net)
- SW25 pad 1: /TM1638 Module/K3 -> (no net)
- SW25 pad 2: /TM1638 Module/K3 -> (no net)
- SW25 pad 3: Net-(D42-Pad1) -> (no net)
- SW26 pad 1: /TM1638 Module/K3 -> (no net)
- SW26 pad 2: /TM1638 Module/K3 -> (no net)
- SW26 pad 3: Net-(D43-Pad1) -> (no net)
- SW27 pad 1: /TM1638 Module/K3 -> (no net)
- SW27 pad 2: /TM1638 Module/K3 -> (no net)
- SW27 pad 3: Net-(D44-Pad1) -> (no net)
- SW28 pad 1: /TM1638 Module/K3 -> (no net)
- SW28 pad 2: /TM1638 Module/K3 -> (no net)
- SW28 pad 3: Net-(D45-Pad1) -> (no net)
- SW29 pad 1: /sheet5C6557AC/K1 -> (no net)
- SW29 pad 2: /sheet5C6557AC/K1 -> (no net)
- SW29 pad 3: Net-(D54-Pad1) -> (no net)
- SW30 pad 1: /sheet5C6557AC/K1 -> (no net)
- SW30 pad 2: /sheet5C6557AC/K1 -> (no net)
- SW30 pad 3: Net-(D55-Pad1) -> (no net)
- SW31 pad 1: /sheet5C6557AC/K1 -> (no net)
- SW31 pad 2: /sheet5C6557AC/K1 -> (no net)
- SW31 pad 3: Net-(D56-Pad1) -> (no net)
- SW32 pad 1: /sheet5C6557AC/K1 -> (no net)
- SW32 pad 2: /sheet5C6557AC/K1 -> (no net)
- SW32 pad 3: Net-(D57-Pad1) -> (no net)
- SW33 pad 1: /sheet5C6557AC/K1 -> (no net)
- SW33 pad 2: /sheet5C6557AC/K1 -> (no net)
- SW33 pad 3: Net-(D66-Pad1) -> (no net)
- SW34 pad 1: /sheet5C6557AC/K1 -> (no net)
- SW34 pad 2: /sheet5C6557AC/K1 -> (no net)
- SW34 pad 3: Net-(D67-Pad1) -> (no net)
- SW35 pad 1: /sheet5C6557AC/K1 -> (no net)
- SW35 pad 2: /sheet5C6557AC/K1 -> (no net)
- SW35 pad 3: Net-(D68-Pad1) -> (no net)
- SW36 pad 1: /sheet5C6557AC/K1 -> (no net)
- SW36 pad 2: /sheet5C6557AC/K1 -> (no net)
- SW36 pad 3: Net-(D69-Pad1) -> (no net)
- SW37 pad 1: /sheet5C6557AC/K2 -> (no net)
- SW37 pad 2: /sheet5C6557AC/K2 -> (no net)
- SW37 pad 3: Net-(D70-Pad1) -> (no net)
- SW38 pad 1: /sheet5C6557AC/K2 -> (no net)
- SW38 pad 2: /sheet5C6557AC/K2 -> (no net)
- SW38 pad 3: Net-(D71-Pad1) -> (no net)
- SW39 pad 1: /sheet5C6557AC/K2 -> (no net)
- SW39 pad 2: /sheet5C6557AC/K2 -> (no net)
- SW39 pad 3: Net-(D72-Pad1) -> (no net)
- SW40 pad 1: /sheet5C6557AC/K2 -> (no net)
- SW40 pad 2: /sheet5C6557AC/K2 -> (no net)
- SW40 pad 3: Net-(D73-Pad1) -> (no net)
- SW41 pad 1: /sheet5C6557AC/K2 -> (no net)
- SW41 pad 2: /sheet5C6557AC/K2 -> (no net)
- SW41 pad 3: Net-(D74-Pad1) -> (no net)
- SW42 pad 1: /sheet5C6557AC/K2 -> (no net)
- SW42 pad 2: /sheet5C6557AC/K2 -> (no net)
- SW42 pad 3: Net-(D75-Pad1) -> (no net)
- SW43 pad 1: /sheet5C6557AC/K2 -> (no net)
- SW43 pad 2: /sheet5C6557AC/K2 -> (no net)
- SW43 pad 3: Net-(D76-Pad1) -> (no net)
- SW44 pad 1: /sheet5C6557AC/K2 -> (no net)
- SW44 pad 2: /sheet5C6557AC/K2 -> (no net)
- SW44 pad 3: Net-(D77-Pad1) -> (no net)
- SW45 pad 1: /sheet5C6557AC/K3 -> (no net)
- SW45 pad 2: /sheet5C6557AC/K3 -> (no net)
- SW45 pad 3: Net-(D78-Pad1) -> (no net)
- SW46 pad 1: /sheet5C6557AC/K3 -> (no net)
- SW46 pad 2: /sheet5C6557AC/K3 -> (no net)
- SW46 pad 3: Net-(D79-Pad1) -> (no net)
- SW47 pad 1: /sheet5C6557AC/K3 -> (no net)
- SW47 pad 2: /sheet5C6557AC/K3 -> (no net)
- SW47 pad 3: Net-(D80-Pad1) -> (no net)
- SW48 pad 1: /sheet5C6557AC/K3 -> (no net)
- SW48 pad 2: /sheet5C6557AC/K3 -> (no net)
- SW48 pad 3: Net-(D81-Pad1) -> (no net)
- SW49 pad 1: /sheet5C6557AC/K3 -> (no net)
- SW49 pad 2: /sheet5C6557AC/K3 -> (no net)
- SW49 pad 3: Net-(D82-Pad1) -> (no net)
- SW5 pad 1: /TM1638 Module/K1 -> (no net)
- SW5 pad 2: /TM1638 Module/K1 -> (no net)
- SW5 pad 3: Net-(D14-Pad1) -> (no net)
- SW50 pad 1: /sheet5C6557AC/K3 -> (no net)
- SW50 pad 2: /sheet5C6557AC/K3 -> (no net)
- SW50 pad 3: Net-(D83-Pad1) -> (no net)
- SW51 pad 1: /sheet5C6557AC/K3 -> (no net)
- SW51 pad 2: /sheet5C6557AC/K3 -> (no net)
- SW51 pad 3: Net-(D84-Pad1) -> (no net)
- SW52 pad 1: /sheet5C6557AC/K3 -> (no net)
- SW52 pad 2: /sheet5C6557AC/K3 -> (no net)
- SW52 pad 3: Net-(D85-Pad1) -> (no net)
- SW53 pad 1: /sheet5C6559D3/K1 -> (no net)
- SW53 pad 2: /sheet5C6559D3/K1 -> (no net)
- SW53 pad 3: Net-(D94-Pad1) -> (no net)
- SW54 pad 1: /sheet5C6559D3/K1 -> (no net)
- SW54 pad 2: /sheet5C6559D3/K1 -> (no net)
- SW54 pad 3: Net-(D95-Pad1) -> (no net)
- SW55 pad 1: /sheet5C6559D3/K1 -> (no net)
- SW55 pad 2: /sheet5C6559D3/K1 -> (no net)
- SW55 pad 3: Net-(D96-Pad1) -> (no net)
- SW56 pad 1: /sheet5C6559D3/K1 -> (no net)
- SW56 pad 2: /sheet5C6559D3/K1 -> (no net)
- SW56 pad 3: Net-(D97-Pad1) -> (no net)
- SW57 pad 1: /sheet5C6559D3/K1 -> (no net)
- SW57 pad 2: /sheet5C6559D3/K1 -> (no net)
- SW57 pad 3: Net-(D106-Pad1) -> (no net)
- SW58 pad 1: /sheet5C6559D3/K1 -> (no net)
- SW58 pad 2: /sheet5C6559D3/K1 -> (no net)
- SW58 pad 3: Net-(D107-Pad1) -> (no net)
- SW59 pad 1: /sheet5C6559D3/K1 -> (no net)
- SW59 pad 2: /sheet5C6559D3/K1 -> (no net)
- SW59 pad 3: Net-(D108-Pad1) -> (no net)
- SW6 pad 1: /TM1638 Module/K1 -> (no net)
- SW6 pad 2: /TM1638 Module/K1 -> (no net)
- SW6 pad 3: Net-(D15-Pad1) -> (no net)
- SW60 pad 1: /sheet5C6559D3/K1 -> (no net)
- SW60 pad 2: /sheet5C6559D3/K1 -> (no net)
- SW60 pad 3: Net-(D109-Pad1) -> (no net)
- SW61 pad 1: /sheet5C6559D3/K2 -> (no net)
- SW61 pad 2: /sheet5C6559D3/K2 -> (no net)
- SW61 pad 3: Net-(D110-Pad1) -> (no net)
- SW62 pad 1: /sheet5C6559D3/K2 -> (no net)
- SW62 pad 2: /sheet5C6559D3/K2 -> (no net)
- SW62 pad 3: Net-(D111-Pad1) -> (no net)
- SW63 pad 1: /sheet5C6559D3/K2 -> (no net)
- SW63 pad 2: /sheet5C6559D3/K2 -> (no net)
- SW63 pad 3: Net-(D112-Pad1) -> (no net)
- SW64 pad 1: /sheet5C6559D3/K2 -> (no net)
- SW64 pad 2: /sheet5C6559D3/K2 -> (no net)
- SW64 pad 3: Net-(D113-Pad1) -> (no net)
- SW65 pad 1: /sheet5C6559D3/K2 -> (no net)
- SW65 pad 2: /sheet5C6559D3/K2 -> (no net)
- SW65 pad 3: Net-(D114-Pad1) -> (no net)
- SW66 pad 1: /sheet5C6559D3/K2 -> (no net)
- SW66 pad 2: /sheet5C6559D3/K2 -> (no net)
- SW66 pad 3: Net-(D115-Pad1) -> (no net)
- SW67 pad 1: /sheet5C6559D3/K2 -> (no net)
- SW67 pad 2: /sheet5C6559D3/K2 -> (no net)
- SW67 pad 3: Net-(D116-Pad1) -> (no net)
- SW68 pad 1: /sheet5C6559D3/K2 -> (no net)
- SW68 pad 2: /sheet5C6559D3/K2 -> (no net)
- SW68 pad 3: Net-(D117-Pad1) -> (no net)
- SW69 pad 1: /sheet5C6559D3/K3 -> (no net)
- SW69 pad 2: /sheet5C6559D3/K3 -> (no net)
- SW69 pad 3: Net-(D118-Pad1) -> (no net)
- SW7 pad 1: /TM1638 Module/K1 -> (no net)
- SW7 pad 2: /TM1638 Module/K1 -> (no net)
- SW7 pad 3: Net-(D16-Pad1) -> (no net)
- SW70 pad 1: /sheet5C6559D3/K3 -> (no net)
- SW70 pad 2: /sheet5C6559D3/K3 -> (no net)
- SW70 pad 3: Net-(D119-Pad1) -> (no net)
- SW71 pad 1: /sheet5C6559D3/K3 -> (no net)
- SW71 pad 2: /sheet5C6559D3/K3 -> (no net)
- SW71 pad 3: Net-(D120-Pad1) -> (no net)
- SW72 pad 1: /sheet5C6559D3/K3 -> (no net)
- SW72 pad 2: /sheet5C6559D3/K3 -> (no net)
- SW72 pad 3: Net-(D121-Pad1) -> (no net)
- SW73 pad 1: /sheet5C6559D3/K3 -> (no net)
- SW73 pad 2: /sheet5C6559D3/K3 -> (no net)
- SW73 pad 3: Net-(D122-Pad1) -> (no net)
- SW74 pad 1: /sheet5C6559D3/K3 -> (no net)
- SW74 pad 2: /sheet5C6559D3/K3 -> (no net)
- SW74 pad 3: Net-(D123-Pad1) -> (no net)
- SW75 pad 1: /sheet5C6559D3/K3 -> (no net)
- SW75 pad 2: /sheet5C6559D3/K3 -> (no net)
- SW75 pad 3: Net-(D124-Pad1) -> (no net)
- SW76 pad 1: /sheet5C6559D3/K3 -> (no net)
- SW76 pad 2: /sheet5C6559D3/K3 -> (no net)
- SW76 pad 3: Net-(D125-Pad1) -> (no net)
- SW8 pad 1: /TM1638 Module/K1 -> (no net)
- SW8 pad 2: /TM1638 Module/K1 -> (no net)
- SW8 pad 3: Net-(D17-Pad1) -> (no net)
- SW9 pad 1: /TM1638 Module/K1 -> (no net)
- SW9 pad 2: /TM1638 Module/K1 -> (no net)
- SW9 pad 3: Net-(D26-Pad1) -> (no net)
- U3 pad 1: /sheet5CD1D363/low-side -> Net-(R119-Pad1)
- U3 pad 2: /sheet5CD14929/low-side -> Net-(Q1-Pad1)
- U3 pad 5: /sheet5CD0BEEF/low-side -> Net-(R121-Pad1)
- U3 pad 6: /Sheet5CCE7B2F/low-side -> Net-(R124-Pad1)
- U5 pad 23: (no net) -> Net-(J6-Pad1)

Commit message: brain board added, bufixes and final board synchronized with schematic
Parts:
- removed the C16 at (249.6, 101.6)
- removed the C7 at (141.6, 119.4)
- removed Q1: 2N7000, Package_TO_SOT_THT:TO-92_Inline
- removed the R119 at (370.0, 87.4)
- removed the R121 at (379.7, 87.4)
- removed the R122 at (370.0, 93.5)
- removed the R123 at (379.7, 90.4)
- removed the R124 at (370.0, 96.5)
- removed the R125 at (379.7, 93.5)
- removed the R126 at (379.7, 96.5)
- removed the R16 at (238.8, 153.7)
- removed the SW14 at (196.4, 307.0)
- removed the SW2 at (67.3, 180.3)
- removed the SW3 at (274.3, 141.0)
- removed the SW4 at (242.6, 141.0)
- removed the U3 at (191.1, 147.3)
- removed the U4 at (165.7, 131.4)
- added C10: 1nF, Capacitor_THT:C_Disc_D8.0mm_W5.0mm_P7.50mm, F.Cu at (84.0, 26.3)
- added C11: 1nF, Capacitor_THT:C_Disc_D8.0mm_W5.0mm_P7.50mm, F.Cu at (76.8, 47.7)
- added C8: 1nF, Capacitor_THT:C_Disc_D8.0mm_W5.0mm_P7.50mm, F.Cu at (95.0, 26.3)
- added C9: 1nF, Capacitor_THT:C_Disc_D8.0mm_W5.0mm_P7.50mm, F.Cu at (76.8, 41.1)
- added D10: 1N4148, Diode_THT:D_DO-35_SOD27_P7.62mm_Horizontal, F.Cu at (98.4, 35.4)
- added D11: 1N4148, Diode_THT:D_DO-35_SOD27_P7.62mm_Horizontal, F.Cu at (98.4, 42.5)
- added D12: 1N4148, Diode_THT:D_DO-35_SOD27_P7.62mm_Horizontal, F.Cu at (105.3, 31.4)
- added D13: 1N4148, Diode_THT:D_DO-35_SOD27_P7.62mm_Horizontal, F.Cu at (87.6, 46.6)
- added D14: 1N4148, Diode_THT:D_DO-35_SOD27_P7.62mm_Horizontal, F.Cu at (87.3, 52.7)
- added D15: 1N4148, Diode_THT:D_DO-35_SOD27_P7.62mm_Horizontal, F.Cu at (98.4, 39.0)
- added D4: 1N4148, Diode_THT:D_DO-35_SOD27_P7.62mm_Horizontal, F.Cu at (76.6, 52.7)
- added D5: 1N4148, Diode_THT:D_DO-35_SOD27_P7.62mm_Horizontal, F.Cu at (87.6, 39.5)
- added D8: 1N4148, Diode_THT:D_DO-35_SOD27_P7.62mm_Horizontal, F.Cu at (87.6, 43.0)
- added D9: 1N4148, Diode_THT:D_DO-35_SOD27_P7.62mm_Horizontal, F.Cu at (105.9, 24.8)
- added J10: free IO, Connector_PinHeader_2.54mm:PinHeader_1x01_P2.54mm_Vertical, F.Cu at (131.4, 38.1)
- added J11: ISP, Connector_PinHeader_2.54mm:PinHeader_2x05_P2.54mm_Vertical, F.Cu at (77.3, 25.4)
- added J12: free IO, Connector_PinHeader_2.54mm:PinHeader_1x01_P2.54mm_Vertical, F.Cu at (128.7, 47.4)
- added J13: free IO, Connector_PinHeader_2.54mm:PinHeader_1x01_P2.54mm_Vertical, F.Cu at (120.4, 53.5)
- added J5: serial debug, Connector_PinHeader_2.54mm:PinHeader_2x01_P2.54mm_Vertical, F.Cu at (131.4, 33.5)
- added J6: +5V, Connector_PinHeader_2.54mm:PinHeader_1x01_P2.54mm_Vertical, F.Cu at (131.4, 42.8)
- added J7: GND, Connector_PinHeader_2.54mm:PinHeader_1x01_P2.54mm_Vertical, F.Cu at (125.0, 53.5)
- added R137: 33, Resistor_THT:R_Axial_DIN0207_L6.3mm_D2.5mm_P10.16mm_Horizontal, F.Cu at (141.2, 44.5)
- added R138: 33, Resistor_THT:R_Axial_DIN0207_L6.3mm_D2.5mm_P10.16mm_Horizontal, F.Cu at (141.2, 48.5)
- added R139: 10k, Resistor_THT:R_Axial_DIN0207_L6.3mm_D2.5mm_P10.16mm_Horizontal, F.Cu at (162.9, 25.1)
- added R140: 33, Resistor_THT:R_Axial_DIN0207_L6.3mm_D2.5mm_P10.16mm_Horizontal, F.Cu at (162.9, 29.1)
- added R141: 33, Resistor_THT:R_Axial_DIN0207_L6.3mm_D2.5mm_P10.16mm_Horizontal, F.Cu at (162.9, 33.2)
- added R142: 33, Resistor_THT:R_Axial_DIN0207_L6.3mm_D2.5mm_P10.16mm_Horizontal, F.Cu at (154.5, 44.5)
- added R143: 33, Resistor_THT:R_Axial_DIN0207_L6.3mm_D2.5mm_P10.16mm_Horizontal, F.Cu at (154.5, 48.5)
- added R144: 33, Resistor_THT:R_Axial_DIN0207_L6.3mm_D2.5mm_P10.16mm_Horizontal, F.Cu at (162.9, 37.2)
- added R145: 33, Resistor_THT:R_Axial_DIN0207_L6.3mm_D2.5mm_P10.16mm_Horizontal, F.Cu at (176.2, 25.1)
- added R18: 10k, Resistor_THT:R_Axial_DIN0207_L6.3mm_D2.5mm_P10.16mm_Horizontal, F.Cu at (109.2, 39.2)
- added R19: 10k, Resistor_THT:R_Axial_DIN0207_L6.3mm_D2.5mm_P10.16mm_Horizontal, F.Cu at (127.4, 25.1)
- added R20: 10k, Resistor_THT:R_Axial_DIN0207_L6.3mm_D2.5mm_P10.16mm_Horizontal, F.Cu at (109.2, 43.3)
- added R21: 10k, Resistor_THT:R_Axial_DIN0207_L6.3mm_D2.5mm_P10.16mm_Horizontal, F.Cu at (119.9, 33.2)
- added R22: 10k, Resistor_THT:R_Axial_DIN0207_L6.3mm_D2.5mm_P10.16mm_Horizontal, F.Cu at (94.5, 31.6)
- added R23: 10k, Resistor_THT:R_Axial_DIN0207_L6.3mm_D2.5mm_P10.16mm_Horizontal, F.Cu at (98.1, 54.4)
- added R24: 10k, Resistor_THT:R_Axial_DIN0207_L6.3mm_D2.5mm_P10.16mm_Horizontal, F.Cu at (126.8, 29.1)
- added R25: 220, Resistor_THT:R_Axial_DIN0207_L6.3mm_D2.5mm_P10.16mm_Horizontal, F.Cu at (108.9, 50.4)
- added R26: 220, Resistor_THT:R_Axial_DIN0207_L6.3mm_D2.5mm_P10.16mm_Horizontal, F.Cu at (119.9, 37.2)
- added R27: 1k, Resistor_THT:R_Axial_DIN0207_L6.3mm_D2.5mm_P10.16mm_Horizontal, F.Cu at (119.9, 41.3)
- added R28: 1k, Resistor_THT:R_Axial_DIN0207_L6.3mm_D2.5mm_P10.16mm_Horizontal, F.Cu at (116.6, 25.1)
- added R29: 1k, Resistor_THT:R_Axial_DIN0207_L6.3mm_D2.5mm_P10.16mm_Horizontal, F.Cu at (108.9, 54.4)
- added R3: 220, Resistor_THT:R_Axial_DIN0207_L6.3mm_D2.5mm_P10.16mm_Horizontal, F.Cu at (109.2, 35.2)
- added R30: 220, Resistor_THT:R_Axial_DIN0207_L6.3mm_D2.5mm_P10.16mm_Horizontal, F.Cu at (83.8, 31.6)
- added R31: 220, Resistor_THT:R_Axial_DIN0207_L6.3mm_D2.5mm_P10.16mm_Horizontal, F.Cu at (87.6, 35.7)
- added R4: 220, Resistor_THT:R_Axial_DIN0207_L6.3mm_D2.5mm_P10.16mm_Horizontal, F.Cu at (98.4, 46.3)
- added R50: 10k, Resistor_THT:R_Axial_DIN0207_L6.3mm_D2.5mm_P10.16mm_Horizontal, F.Cu at (76.6, 62.8)
- added R85: 10k, Resistor_THT:R_Axial_DIN0207_L6.3mm_D2.5mm_P10.16mm_Horizontal, F.Cu at (141.2, 55.6)
- added SW11: SW_Push, beat707:B3F-through-hole, F.Cu at (67.3, 180.5)
- added U13: SN74AHC125, Package_DIP:DIP-14_W7.62mm, F.Cu at (141.3, 25.1)
- added U14: MB85RS2MT, Package_DIP:DIP-8_W7.62mm, F.Cu at (176.3, 29.2)
- added U15: LP2950CZ-3.3G, Package_TO_SOT_THT:TO-92_Inline, F.Cu at (168.3, 42.5)
- added U16: SN74AHCT125, Package_DIP:DIP-14_W7.62mm, F.Cu at (152.1, 25.1)
- C15: renamed from C12; value 10uF -> 100nF; footprint Capacitor_THT:CP_Radial_D6.3mm_P2.50mm -> Capacitor_THT:C_Disc_D3.0mm_W2.0mm_P2.50mm
- C17: renamed from C14; value 10uF -> 100nF; footprint Capacitor_THT:CP_Radial_D6.3mm_P2.50mm -> Capacitor_THT:C_Disc_D3.0mm_W2.0mm_P2.50mm
- C5: value 100nF -> 47uF; footprint Capacitor_THT:C_Disc_D3.0mm_W2.0mm_P2.50mm -> Capacitor_THT:CP_Radial_D6.3mm_P2.50mm
- R1, R14, R15, R2: footprint Resistor_THT:R_Axial_DIN0207_L6.3mm_D2.5mm_P7.62mm_Horizontal -> Resistor_THT:R_Axial_DIN0207_L6.3mm_D2.5mm_P10.16mm_Horizontal
- R10: renamed from R8; footprint Resistor_THT:R_Axial_DIN0207_L6.3mm_D2.5mm_P7.62mm_Horizontal -> Resistor_THT:R_Axial_DIN0207_L6.3mm_D2.5mm_P10.16mm_Horizontal
- R100: renamed from R83; footprint Resistor_THT:R_Axial_DIN0207_L6.3mm_D2.5mm_P7.62mm_Horizontal -> Resistor_THT:R_Axial_DIN0207_L6.3mm_D2.5mm_P10.16mm_Horizontal
- R101: renamed from R84; footprint Resistor_THT:R_Axial_DIN0207_L6.3mm_D2.5mm_P7.62mm_Horizontal -> Resistor_THT:R_Axial_DIN0207_L6.3mm_D2.5mm_P10.16mm_Horizontal
- R102: renamed from R85; footprint Resistor_THT:R_Axial_DIN0207_L6.3mm_D2.5mm_P7.62mm_Horizontal -> Resistor_THT:R_Axial_DIN0207_L6.3mm_D2.5mm_P10.16mm_Horizontal
- R103: renamed from R86; footprint Resistor_THT:R_Axial_DIN0207_L6.3mm_D2.5mm_P7.62mm_Horizontal -> Resistor_THT:R_Axial_DIN0207_L6.3mm_D2.5mm_P10.16mm_Horizontal
- R104: renamed from R87; footprint Resistor_THT:R_Axial_DIN0207_L6.3mm_D2.5mm_P7.62mm_Horizontal -> Resistor_THT:R_Axial_DIN0207_L6.3mm_D2.5mm_P10.16mm_Horizontal
- R105: renamed from R88; footprint Resistor_THT:R_Axial_DIN0207_L6.3mm_D2.5mm_P7.62mm_Horizontal -> Resistor_THT:R_Axial_DIN0207_L6.3mm_D2.5mm_P10.16mm_Horizontal
- R106: renamed from R89; footprint Resistor_THT:R_Axial_DIN0207_L6.3mm_D2.5mm_P7.62mm_Horizontal -> Resistor_THT:R_Axial_DIN0207_L6.3mm_D2.5mm_P10.16mm_Horizontal
- R107: renamed from R90; footprint Resistor_THT:R_Axial_DIN0207_L6.3mm_D2.5mm_P7.62mm_Horizontal -> Resistor_THT:R_Axial_DIN0207_L6.3mm_D2.5mm_P10.16mm_Horizontal
- R108: renamed from R91; footprint Resistor_THT:R_Axial_DIN0207_L6.3mm_D2.5mm_P7.62mm_Horizontal -> Resistor_THT:R_Axial_DIN0207_L6.3mm_D2.5mm_P10.16mm_Horizontal
- R109: renamed from R92; footprint Resistor_THT:R_Axial_DIN0207_L6.3mm_D2.5mm_P7.62mm_Horizontal -> Resistor_THT:R_Axial_DIN0207_L6.3mm_D2.5mm_P10.16mm_Horizontal
- R11: renamed from R9; footprint Resistor_THT:R_Axial_DIN0207_L6.3mm_D2.5mm_P7.62mm_Horizontal -> Resistor_THT:R_Axial_DIN0207_L6.3mm_D2.5mm_P10.16mm_Horizontal
- R110: renamed from R93; footprint Resistor_THT:R_Axial_DIN0207_L6.3mm_D2.5mm_P7.62mm_Horizontal -> Resistor_THT:R_Axial_DIN0207_L6.3mm_D2.5mm_P10.16mm_Horizontal
- R111: renamed from R94; footprint Resistor_THT:R_Axial_DIN0207_L6.3mm_D2.5mm_P7.62mm_Horizontal -> Resistor_THT:R_Axial_DIN0207_L6.3mm_D2.5mm_P10.16mm_Horizontal
- R112: renamed from R95; footprint Resistor_THT:R_Axial_DIN0207_L6.3mm_D2.5mm_P7.62mm_Horizontal -> Resistor_THT:R_Axial_DIN0207_L6.3mm_D2.5mm_P10.16mm_Horizontal
- R113: renamed from R96; footprint Resistor_THT:R_Axial_DIN0207_L6.3mm_D2.5mm_P7.62mm_Horizontal -> Resistor_THT:R_Axial_DIN0207_L6.3mm_D2.5mm_P10.16mm_Horizontal
- R114: renamed from R97; footprint Resistor_THT:R_Axial_DIN0207_L6.3mm_D2.5mm_P7.62mm_Horizontal -> Resistor_THT:R_Axial_DIN0207_L6.3mm_D2.5mm_P10.16mm_Horizontal
- R115: renamed from R98; footprint Resistor_THT:R_Axial_DIN0207_L6.3mm_D2.5mm_P7.62mm_Horizontal -> Resistor_THT:R_Axial_DIN0207_L6.3mm_D2.5mm_P10.16mm_Horizontal
- R116: renamed from R99; footprint Resistor_THT:R_Axial_DIN0207_L6.3mm_D2.5mm_P7.62mm_Horizontal -> Resistor_THT:R_Axial_DIN0207_L6.3mm_D2.5mm_P10.16mm_Horizontal
- R117: renamed from R100; footprint Resistor_THT:R_Axial_DIN0207_L6.3mm_D2.5mm_P7.62mm_Horizontal -> Resistor_THT:R_Axial_DIN0207_L6.3mm_D2.5mm_P10.16mm_Horizontal
- R118: renamed from R101; footprint Resistor_THT:R_Axial_DIN0207_L6.3mm_D2.5mm_P7.62mm_Horizontal -> Resistor_THT:R_Axial_DIN0207_L6.3mm_D2.5mm_P10.16mm_Horizontal
- R119: renamed from R102; footprint Resistor_THT:R_Axial_DIN0207_L6.3mm_D2.5mm_P7.62mm_Horizontal -> Resistor_THT:R_Axial_DIN0207_L6.3mm_D2.5mm_P10.16mm_Horizontal
- R12: renamed from R10; footprint Resistor_THT:R_Axial_DIN0207_L6.3mm_D2.5mm_P7.62mm_Horizontal -> Resistor_THT:R_Axial_DIN0207_L6.3mm_D2.5mm_P10.16mm_Horizontal
- R120: value 3.3k -> 10k; footprint Resistor_THT:R_Axial_DIN0207_L6.3mm_D2.5mm_P7.62mm_Horizontal -> Resistor_THT:R_Axial_DIN0207_L6.3mm_D2.5mm_P10.16mm_Horizontal
- R121: renamed from R103; footprint Resistor_THT:R_Axial_DIN0207_L6.3mm_D2.5mm_P7.62mm_Horizontal -> Resistor_THT:R_Axial_DIN0207_L6.3mm_D2.5mm_P10.16mm_Horizontal
- R122: renamed from R104; footprint Resistor_THT:R_Axial_DIN0207_L6.3mm_D2.5mm_P7.62mm_Horizontal -> Resistor_THT:R_Axial_DIN0207_L6.3mm_D2.5mm_P10.16mm_Horizontal
- R123: renamed from R105; footprint Resistor_THT:R_Axial_DIN0207_L6.3mm_D2.5mm_P7.62mm_Horizontal -> Resistor_THT:R_Axial_DIN0207_L6.3mm_D2.5mm_P10.16mm_Horizontal
- R124: renamed from R106; footprint Resistor_THT:R_Axial_DIN0207_L6.3mm_D2.5mm_P7.62mm_Horizontal -> Resistor_THT:R_Axial_DIN0207_L6.3mm_D2.5mm_P10.16mm_Horizontal
- R125: renamed from R107; footprint Resistor_THT:R_Axial_DIN0207_L6.3mm_D2.5mm_P7.62mm_Horizontal -> Resistor_THT:R_Axial_DIN0207_L6.3mm_D2.5mm_P10.16mm_Horizontal
- R126: renamed from R108; footprint Resistor_THT:R_Axial_DIN0207_L6.3mm_D2.5mm_P7.62mm_Horizontal -> Resistor_THT:R_Axial_DIN0207_L6.3mm_D2.5mm_P10.16mm_Horizontal
- R127: renamed from R109; footprint Resistor_THT:R_Axial_DIN0207_L6.3mm_D2.5mm_P7.62mm_Horizontal -> Resistor_THT:R_Axial_DIN0207_L6.3mm_D2.5mm_P10.16mm_Horizontal
- R128: renamed from R110; footprint Resistor_THT:R_Axial_DIN0207_L6.3mm_D2.5mm_P7.62mm_Horizontal -> Resistor_THT:R_Axial_DIN0207_L6.3mm_D2.5mm_P10.16mm_Horizontal
- R129: renamed from R111; footprint Resistor_THT:R_Axial_DIN0207_L6.3mm_D2.5mm_P7.62mm_Horizontal -> Resistor_THT:R_Axial_DIN0207_L6.3mm_D2.5mm_P10.16mm_Horizontal
- R13: renamed from R11; footprint Resistor_THT:R_Axial_DIN0207_L6.3mm_D2.5mm_P7.62mm_Horizontal -> Resistor_THT:R_Axial_DIN0207_L6.3mm_D2.5mm_P10.16mm_Horizontal
- R130: renamed from R112; footprint Resistor_THT:R_Axial_DIN0207_L6.3mm_D2.5mm_P7.62mm_Horizontal -> Resistor_THT:R_Axial_DIN0207_L6.3mm_D2.5mm_P10.16mm_Horizontal
- R131: renamed from R113; footprint Resistor_THT:R_Axial_DIN0207_L6.3mm_D2.5mm_P7.62mm_Horizontal -> Resistor_THT:R_Axial_DIN0207_L6.3mm_D2.5mm_P10.16mm_Horizontal
- R132: renamed from R114; footprint Resistor_THT:R_Axial_DIN0207_L6.3mm_D2.5mm_P7.62mm_Horizontal -> Resistor_THT:R_Axial_DIN0207_L6.3mm_D2.5mm_P10.16mm_Horizontal
- R133: renamed from R115; footprint Resistor_THT:R_Axial_DIN0207_L6.3mm_D2.5mm_P7.62mm_Horizontal -> Resistor_THT:R_Axial_DIN0207_L6.3mm_D2.5mm_P10.16mm_Horizontal
- R134: renamed from R116; footprint Resistor_THT:R_Axial_DIN0207_L6.3mm_D2.5mm_P7.62mm_Horizontal -> Resistor_THT:R_Axial_DIN0207_L6.3mm_D2.5mm_P10.16mm_Horizontal
- R135: renamed from R117; footprint Resistor_THT:R_Axial_DIN0207_L6.3mm_D2.5mm_P7.62mm_Horizontal -> Resistor_THT:R_Axial_DIN0207_L6.3mm_D2.5mm_P10.16mm_Horizontal
- R136: renamed from R118; footprint Resistor_THT:R_Axial_DIN0207_L6.3mm_D2.5mm_P7.62mm_Horizontal -> Resistor_THT:R_Axial_DIN0207_L6.3mm_D2.5mm_P10.16mm_Horizontal
- R16: renamed from R13; footprint Resistor_THT:R_Axial_DIN0207_L6.3mm_D2.5mm_P7.62mm_Horizontal -> Resistor_THT:R_Axial_DIN0207_L6.3mm_D2.5mm_P10.16mm_Horizontal
- R17: renamed from R12; footprint Resistor_THT:R_Axial_DIN0207_L6.3mm_D2.5mm_P7.62mm_Horizontal -> Resistor_THT:R_Axial_DIN0207_L6.3mm_D2.5mm_P10.16mm_Horizontal
- R32: renamed from R17; footprint Resistor_THT:R_Axial_DIN0207_L6.3mm_D2.5mm_P7.62mm_Horizontal -> Resistor_THT:R_Axial_DIN0207_L6.3mm_D2.5mm_P10.16mm_Horizontal
- R33: renamed from R18; footprint Resistor_THT:R_Axial_DIN0207_L6.3mm_D2.5mm_P7.62mm_Horizontal -> Resistor_THT:R_Axial_DIN0207_L6.3mm_D2.5mm_P10.16mm_Horizontal
- R34: renamed from R19; footprint Resistor_THT:R_Axial_DIN0207_L6.3mm_D2.5mm_P7.62mm_Horizontal -> Resistor_THT:R_Axial_DIN0207_L6.3mm_D2.5mm_P10.16mm_Horizontal
- R35: renamed from R20; footprint Resistor_THT:R_Axial_DIN0207_L6.3mm_D2.5mm_P7.62mm_Horizontal -> Resistor_THT:R_Axial_DIN0207_L6.3mm_D2.5mm_P10.16mm_Horizontal
- R36: renamed from R21; footprint Resistor_THT:R_Axial_DIN0207_L6.3mm_D2.5mm_P7.62mm_Horizontal -> Resistor_THT:R_Axial_DIN0207_L6.3mm_D2.5mm_P10.16mm_Horizontal
- R37: renamed from R22; footprint Resistor_THT:R_Axial_DIN0207_L6.3mm_D2.5mm_P7.62mm_Horizontal -> Resistor_THT:R_Axial_DIN0207_L6.3mm_D2.5mm_P10.16mm_Horizontal
- R38: renamed from R23; footprint Resistor_THT:R_Axial_DIN0207_L6.3mm_D2.5mm_P7.62mm_Horizontal -> Resistor_THT:R_Axial_DIN0207_L6.3mm_D2.5mm_P10.16mm_Horizontal
- R39: renamed from R24; footprint Resistor_THT:R_Axial_DIN0207_L6.3mm_D2.5mm_P7.62mm_Horizontal -> Resistor_THT:R_Axial_DIN0207_L6.3mm_D2.5mm_P10.16mm_Horizontal
- R40: renamed from R25; footprint Resistor_THT:R_Axial_DIN0207_L6.3mm_D2.5mm_P7.62mm_Horizontal -> Resistor_THT:R_Axial_DIN0207_L6.3mm_D2.5mm_P10.16mm_Horizontal
- R41: renamed from R26; footprint Resistor_THT:R_Axial_DIN0207_L6.3mm_D2.5mm_P7.62mm_Horizontal -> Resistor_THT:R_Axial_DIN0207_L6.3mm_D2.5mm_P10.16mm_Horizontal
- R42: renamed from R27; footprint Resistor_THT:R_Axial_DIN0207_L6.3mm_D2.5mm_P7.62mm_Horizontal -> Resistor_THT:R_Axial_DIN0207_L6.3mm_D2.5mm_P10.16mm_Horizontal
- R43: renamed from R28; footprint Resistor_THT:R_Axial_DIN0207_L6.3mm_D2.5mm_P7.62mm_Horizontal -> Resistor_THT:R_Axial_DIN0207_L6.3mm_D2.5mm_P10.16mm_Horizontal
- R44: renamed from R29; footprint Resistor_THT:R_Axial_DIN0207_L6.3mm_D2.5mm_P7.62mm_Horizontal -> Resistor_THT:R_Axial_DIN0207_L6.3mm_D2.5mm_P10.16mm_Horizontal
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- renumbered C9 to C12, C10 to C13, C11 to C14, C13 to C16, C15 to C18, C8 to C6, C6 to C7, D90 to D100, D91 to D101, D92 to D102, D93 to D103, D94 to D104, D95 to D105, D96 to D106, D97 to D107, D98 to D108, D99 to D109, D100 to D110, D101 to D111, D102 to D112, D103 to D113, D104 to D114, D105 to D115, D106 to D116, D107 to D117, D108 to D118, D109 to D119, D110 to D120, D111 to D121, D112 to D122, D113 to D123, D114 to D124, D115 to D125, D116 to D126, D117 to D127, D118 to D128, D119 to D129, D120 to D130, D121 to D131, D122 to D132, D123 to D133, D124 to D134, D125 to D135, D6 to D16, D7 to D17, D8 to D18, D9 to D19, D10 to D20, D11 to D21, D12 to D22, D13 to D23, D14 to D24, D15 to D25, D16 to D26, D17 to D27, D18 to D28, D19 to D29, D20 to D30, D21 to D31, D22 to D32, D23 to D33, D24 to D34, D25 to D35, D26 to D36, D27 to D37, D28 to D38, D29 to D39, D30 to D40, D31 to D41, D32 to D42, D33 to D43, D34 to D44, D35 to D45, D36 to D46, D37 to D47, D38 to D48, D39 to D49, D40 to D50, D41 to D51, D42 to D52, D43 to D53, D44 to D54, D45 to D55, D46 to D56, D47 to D57, D48 to D58, D49 to D59, D4 to D6, D50 to D60, D51 to D61, D52 to D62, D53 to D63, D54 to D64, D55 to D65, D56 to D66, D57 to D67, D58 to D68, D59 to D69, D5 to D7, D60 to D70, D61 to D71, D62 to D72, D63 to D73, D64 to D74, D65 to D75, D66 to D76, D67 to D77, D68 to D78, D69 to D79, D70 to D80, D71 to D81, D72 to D82, D73 to D83, D74 to D84, D75 to D85, D76 to D86, D77 to D87, D78 to D88, D79 to D89, D80 to D90, D81 to D91, D82 to D92, D83 to D93, D84 to D94, D85 to D95, D86 to D96, D87 to D97, D88 to D98, D89 to D99, J5 to J8, J6 to J9, SW13 to SW10, SW15 to SW12, SW16 to SW13, SW17 to SW14, SW18 to SW15, SW19 to SW16, SW20 to SW17, SW21 to SW18, SW22 to SW19, SW5 to SW2, SW23 to SW20, SW24 to SW21, SW25 to SW22, SW26 to SW23, SW27 to SW24, SW28 to SW25, SW29 to SW26, SW30 to SW27, SW31 to SW28, SW32 to SW29, SW6 to SW3, SW33 to SW30, SW34 to SW31, SW35 to SW32, SW36 to SW33, SW37 to SW34, SW38 to SW35, SW39 to SW36, SW40 to SW37, SW41 to SW38, SW42 to SW39, SW7 to SW4, SW43 to SW40, SW44 to SW41, SW45 to SW42, SW46 to SW43, SW47 to SW44, SW48 to SW45, SW49 to SW46, SW50 to SW47, SW51 to SW48, SW52 to SW49, SW8 to SW5, SW53 to SW50, SW54 to SW51, SW55 to SW52, SW56 to SW53, SW57 to SW54, SW58 to SW55, SW59 to SW56, SW60 to SW57, SW61 to SW58, SW62 to SW59, SW9 to SW6, SW63 to SW60, SW64 to SW61, SW65 to SW62, SW66 to SW63, SW67 to SW64, SW68 to SW65, SW69 to SW66, SW70 to SW67, SW71 to SW68, SW72 to SW69, SW10 to SW7, SW73 to SW70, SW74 to SW71, SW75 to SW72, SW76 to SW73, SW11 to SW8, SW12 to SW9, U12 to U10, U13 to U11, U14 to U12, U5 to U3, U6 to U4, U7 to U5, U8 to U6, U9 to U7, U10 to U8, U11 to U9
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Connections:
- C18 pad 1: +5V -> GND
- C18 pad 2: GND -> +3V3
- C5 pad 1: GND -> +5V
- C5 pad 2: +3V3 -> GND
- C7 pad 2: GND -> Net-(C7-Pad2)
- D105 pad 2: /sheet5C6559D3/SEG2 -> /sheet5C6559D3/SEG3
- D106 pad 2: /sheet5C6559D3/SEG3 -> /sheet5C6559D3/SEG5
- D107 pad 2: /sheet5C6559D3/SEG4 -> /sheet5C6559D3/SEG7
- D116 pad 2: /sheet5C6559D3/SEG5 -> /sheet5C6559D3/SEG2
- D117 pad 2: /sheet5C6559D3/SEG6 -> /sheet5C6559D3/SEG4
- D118 pad 2: /sheet5C6559D3/SEG7 -> /sheet5C6559D3/SEG6
- D121 pad 2: /sheet5C6559D3/SEG2 -> /sheet5C6559D3/SEG3
- D122 pad 2: /sheet5C6559D3/SEG3 -> /sheet5C6559D3/SEG5
- D123 pad 2: /sheet5C6559D3/SEG4 -> /sheet5C6559D3/SEG7
- D124 pad 2: /sheet5C6559D3/SEG5 -> /sheet5C6559D3/SEG2
- D125 pad 2: /sheet5C6559D3/SEG6 -> /sheet5C6559D3/SEG4
- D126 pad 2: /sheet5C6559D3/SEG7 -> /sheet5C6559D3/SEG6
- D129 pad 2: /sheet5C6559D3/SEG2 -> /sheet5C6559D3/SEG3
- D130 pad 2: /sheet5C6559D3/SEG3 -> /sheet5C6559D3/SEG5
- D131 pad 2: /sheet5C6559D3/SEG4 -> /sheet5C6559D3/SEG7
- D132 pad 2: /sheet5C6559D3/SEG5 -> /sheet5C6559D3/SEG2
- D133 pad 2: /sheet5C6559D3/SEG6 -> /sheet5C6559D3/SEG4
- D134 pad 2: /sheet5C6559D3/SEG7 -> /sheet5C6559D3/SEG6
- D25 pad 2: /TM1638 Module/SEG2 -> /TM1638 Module/SEG3
- D26 pad 2: /TM1638 Module/SEG3 -> /TM1638 Module/SEG5
- D27 pad 2: /TM1638 Module/SEG4 -> /TM1638 Module/SEG7
- D36 pad 2: /TM1638 Module/SEG5 -> /TM1638 Module/SEG2
- D37 pad 2: /TM1638 Module/SEG6 -> /TM1638 Module/SEG4
- D38 pad 2: /TM1638 Module/SEG7 -> /TM1638 Module/SEG6
- D41 pad 2: /TM1638 Module/SEG2 -> /TM1638 Module/SEG3
- D42 pad 2: /TM1638 Module/SEG3 -> /TM1638 Module/SEG5
- D43 pad 2: /TM1638 Module/SEG4 -> /TM1638 Module/SEG7
- D44 pad 2: /TM1638 Module/SEG5 -> /TM1638 Module/SEG2
- D45 pad 2: /TM1638 Module/SEG6 -> /TM1638 Module/SEG4
- D46 pad 2: /TM1638 Module/SEG7 -> /TM1638 Module/SEG6
- D49 pad 2: /TM1638 Module/SEG2 -> /TM1638 Module/SEG3
- D50 pad 2: /TM1638 Module/SEG3 -> /TM1638 Module/SEG5
- D51 pad 2: /TM1638 Module/SEG4 -> /TM1638 Module/SEG7
- D52 pad 2: /TM1638 Module/SEG5 -> /TM1638 Module/SEG2
- D53 pad 2: /TM1638 Module/SEG6 -> /TM1638 Module/SEG4
- D54 pad 2: /TM1638 Module/SEG7 -> /TM1638 Module/SEG6
- D65 pad 2: /sheet5C6557AC/SEG2 -> /sheet5C6557AC/SEG3
- D66 pad 2: /sheet5C6557AC/SEG3 -> /sheet5C6557AC/SEG5
- D67 pad 2: /sheet5C6557AC/SEG4 -> /sheet5C6557AC/SEG7
- D76 pad 2: /sheet5C6557AC/SEG5 -> /sheet5C6557AC/SEG2
- D77 pad 2: /sheet5C6557AC/SEG6 -> /sheet5C6557AC/SEG4
- D78 pad 2: /sheet5C6557AC/SEG7 -> /sheet5C6557AC/SEG6
- D81 pad 2: /sheet5C6557AC/SEG2 -> /sheet5C6557AC/SEG3
- D82 pad 2: /sheet5C6557AC/SEG3 -> /sheet5C6557AC/SEG5
- D83 pad 2: /sheet5C6557AC/SEG4 -> /sheet5C6557AC/SEG7
- D84 pad 2: /sheet5C6557AC/SEG5 -> /sheet5C6557AC/SEG2
- D85 pad 2: /sheet5C6557AC/SEG6 -> /sheet5C6557AC/SEG4
- D86 pad 2: /sheet5C6557AC/SEG7 -> /sheet5C6557AC/SEG6
- D89 pad 2: /sheet5C6557AC/SEG2 -> /sheet5C6557AC/SEG3
- D90 pad 2: /sheet5C6557AC/SEG3 -> /sheet5C6557AC/SEG5
- D91 pad 2: /sheet5C6557AC/SEG4 -> /sheet5C6557AC/SEG7
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
Commit message: mounting holes and all parts placed
Parts:
- added H1: MountingHole, MountingHole:MountingHole_3.2mm_M3, F.Cu at (142.2, 231.1)
- added H10: MountingHole, MountingHole:MountingHole_3.2mm_M3, F.Cu at (320.0, 231.1)
- added H11: MountingHole, MountingHole:MountingHole_3.2mm_M3, F.Cu at (53.3, 231.1)
- added H12: MountingHole, MountingHole:MountingHole_3.2mm_M3, F.Cu at (53.3, 99.1)
- added H2: MountingHole, MountingHole:MountingHole_3.2mm_M3, F.Cu at (231.1, 231.1)
- added H3: MountingHole, MountingHole:MountingHole_3.2mm_M3, F.Cu at (142.2, 165.1)
- added H4: MountingHole, MountingHole:MountingHole_3.2mm_M3, F.Cu at (320.0, 165.1)
- added H5: MountingHole, MountingHole:MountingHole_3.2mm_M3, F.Cu at (228.6, 165.1)
- added H6: MountingHole, MountingHole:MountingHole_3.2mm_M3, F.Cu at (142.2, 99.1)
- added H7: MountingHole, MountingHole:MountingHole_3.2mm_M3, F.Cu at (53.3, 165.1)
- added H8: MountingHole, MountingHole:MountingHole_3.2mm_M3, F.Cu at (231.1, 99.1)
- added H9: MountingHole, MountingHole:MountingHole_3.2mm_M3, F.Cu at (320.0, 99.1)
- U10, U4, U7: moved to B.Cu
- moved J9 246.0 mm to (144.8, 108.0)
- moved R30 184.6 mm to (209.7, 166.7), turned to 90 degrees
- moved R137 183.0 mm to (301.3, 133.3)
- moved D8 179.4 mm to (221.1, 162.8), turned to 90 degrees
- moved D5 179.2 mm to (217.5, 162.8), turned to 90 degrees
- moved R31 179.1 mm to (213.7, 162.8), turned to 90 degrees
- moved C10 178.9 mm to (189.2, 170.9), turned to 90 degrees
- moved D14 177.9 mm to (231.1, 157.5), turned to 90 degrees
- moved D13 177.9 mm to (224.6, 160.0), turned to 90 degrees
- moved C9 161.1 mm to (172.2, 170.9), turned to 90 degrees
- moved C11 159.9 mm to (178.8, 170.9), turned to 90 degrees
- moved D4 159.7 mm to (183.8, 171.1), turned to 90 degrees
- moved R50 159.7 mm to (203.2, 160.0), turned to 90 degrees
- moved R145 155.4 mm to (66.0, 134.6)
- moved R20 149.2 mm to (215.9, 147.6)
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Other:
- board size 274.3 x 134.6 mm -> 276.9 x 142.2 mm

Commit message: 5 new menu buttons
Parts:
- moved SW41 213.6 mm to (200.7, 159.9), turned to 90 degrees
- moved SW34 194.1 mm to (182.9, 160.0), turned to 90 degrees
- moved SW59 185.2 mm to (214.6, 160.0), turned to 90 degrees
- moved R79 185.2 mm to (149.9, 170.2)
- moved R84 176.7 mm to (195.6, 170.2)
- moved SW36 176.0 mm to (154.9, 160.0), turned to 90 degrees
- moved SW40 175.2 mm to (168.9, 160.0), turned to 90 degrees
- moved D86 172.3 mm to (165.1, 170.2)
- moved D10 171.8 mm to (315.4, 147.5)
- moved D15 171.8 mm to (318.9, 147.5)
- moved R22 171.8 mm to (311.1, 149.9)
- moved R113 162.0 mm to (209.6, 170.2)
- moved D80 156.6 mm to (179.1, 170.2)
- moved R4 139.2 mm to (293.4, 186.7)
- moved C8 121.4 mm to (52.1, 129.5)
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Other:
- board text added: "BANK OPTIONS"
- board text added: "NEXT"
- board text added: "PATTERN OPTIONS"
- board text added: "PREVIOUS"
- board text added: "TRACK OPTIONS"
