File: kicad/beat707/tm1638-module.sch (KiCad schematic (older format))
At the start: 18 parts, among them SW1 SW_Push, SW2 SW_Push, SW3 SW_Push, SW4 SW_Push, SW5 SW_Push, SW6 SW_Push, SW7 SW_Push, SW8 SW_Push, U2 CA56-12EWA, U3 CA56-12EWA

Commit message: all LEDs changed to through-hole, 3mm
Parts:
- D1, D2, D3, D4, D5, D6, D7, D8: footprint LED_SMD:LED_0603_1608Metric_Castellated -> LED_THT:LED_D3.0mm
Changed lines of the file:
@@
 F 0 "D1" H 3791 2766 50  0000 C CNN
 F 1 "LED" H 3791 2675 50  0000 C CNN
-F 2 "LED_SMD:LED_0603_1608Metric_Castellated" H 3800 2550 50  0001 C CNN
+F 2 "LED_THT:LED_D3.0mm" H 3800 2550 50  0001 C CNN
 F 3 "~" H 3800 2550 50  0001 C CNN
 	1    3800 2550
@@
 F 0 "D2" H 3791 3216 50  0000 C CNN
 F 1 "LED" H 3791 3125 50  0000 C CNN
-F 2 "LED_SMD:LED_0603_1608Metric_Castellated" H 3800 3000 50  0001 C CNN
+F 2 "LED_THT:LED_D3.0mm" H 3800 3000 50  0001 C CNN
 F 3 "~" H 3800 3000 50  0001 C CNN
 	1    3800 3000
@@
 F 0 "D3" H 3791 3966 50  0000 C CNN
 F 1 "LED" H 3791 3875 50  0000 C CNN
-F 2 "LED_SMD:LED_0603_1608Metric_Castellated" H 3800 3750 50  0001 C CNN
+F 2 "LED_THT:LED_D3.0mm" H 3800 3750 50  0001 C CNN
 F 3 "~" H 3800 3750 50  0001 C CNN
 	1    3800 3750
@@
 F 0 "D4" H 3791 4416 50  0000 C CNN
 F 1 "LED" H 3791 4325 50  0000 C CNN
-F 2 "LED_SMD:LED_0603_1608Metric_Castellated" H 3800 4200 50  0001 C CNN
+F 2 "LED_THT:LED_D3.0mm" H 3800 4200 50  0001 C CNN
 F 3 "~" H 3800 4200 50  0001 C CNN
 	1    3800 4200
@@
 F 0 "D5" H 3791 5216 50  0000 C CNN
 F 1 "LED" H 3791 5125 50  0000 C CNN
-F 2 "LED_SMD:LED_0603_1608Metric_Castellated" H 3800 5000 50  0001 C CNN
+F 2 "LED_THT:LED_D3.0mm" H 3800 5000 50  0001 C CNN
 F 3 "~" H 3800 5000 50  0001 C CNN
 	1    3800 5000
@@
 F 0 "D6" H 3791 5666 50  0000 C CNN
 F 1 "LED" H 3791 5575 50  0000 C CNN
-F 2 "LED_SMD:LED_0603_1608Metric_Castellated" H 3800 5450 50  0001 C CNN
+F 2 "LED_THT:LED_D3.0mm" H 3800 5450 50  0001 C CNN
 F 3 "~" H 3800 5450 50  0001 C CNN
 	1    3800 5450
@@
 F 0 "D7" H 3791 6416 50  0000 C CNN
 F 1 "LED" H 3791 6325 50  0000 C CNN
-F 2 "LED_SMD:LED_0603_1608Metric_Castellated" H 3800 6200 50  0001 C CNN
+F 2 "LED_THT:LED_D3.0mm" H 3800 6200 50  0001 C CNN
 F 3 "~" H 3800 6200 50  0001 C CNN
 	1    3800 6200
@@
 F 0 "D8" H 3791 6866 50  0000 C CNN
 F 1 "LED" H 3791 6775 50  0000 C CNN
-F 2 "LED_SMD:LED_0603_1608Metric_Castellated" H 3800 6650 50  0001 C CNN
+F 2 "LED_THT:LED_D3.0mm" H 3800 6650 50  0001 C CNN
 F 3 "~" H 3800 6650 50  0001 C CNN
 	1    3800 6650

Commit message: more LEDs, switches and resistors for version encoding
Parts:
- added C1: 100nF, Capacitor_SMD:C_0805_2012Metric, symbol Device:C
- added C2: 10uF, Capacitor_SMD:C_0805_2012Metric, symbol Device:C
- added D13, D14, D15, D16, D17, D18, D19, D20: LED, LED_THT:LED_D3.0mm, symbol Device:LED
- added D49, D50, D51, D52, D61, D62, D63, D64, D65, D66, D67, D68, D69, D70, D71, D72, D73, D74, D75, D76, D77, D78, D79, D80: 1N4148, Diode_THT:D_DO-35_SOD27_P7.62mm_Horizontal, symbol Diode:1N4148
- added R35, R36, R37, R38, R39, R40, R41, R42, R45, R46, R47, R48, R49, R50, R51, R52, R61, R62, R63, R64, R65, R66, R67, R68: 0, Resistor_THT:R_Axial_DIN0207_L6.3mm_D2.5mm_P7.62mm_Horizontal, symbol Device:R
- added R43, R44, R53, R54, R55, R56, R57, R58, R59, R60: 51, Resistor_THT:R_Axial_DIN0207_L6.3mm_D2.5mm_P7.62mm_Horizontal, symbol Device:R
- added SW13, SW14, SW15, SW16, SW17, SW18, SW19, SW20, SW21, SW22, SW23, SW24, SW25, SW26, SW27, SW28: SW_Push, beat707:K2-1103SP-A4SW-04, symbol switch:SW_Push
- added U2: TM1638, Package_SO:SOIC-28W_7.5x17.9mm_P1.27mm, symbol beat707:TM1638
- renumbered SW6 to SW10, SW7 to SW11, SW8 to SW12, SW1 to SW5, SW2 to SW6, SW3 to SW7, SW4 to SW8, SW5 to SW9, U2 to U3, U3 to U4
Connections:
- net labels added: +5V, CLK, DIO, GND, GRID1, GRID2, GRID3, GRID4, GRID5, GRID6, GRID7, GRID8, K1, K2, K3, SEG1, SEG2, SEG3, SEG4, SEG5, SEG6, SEG7, SEG8, STB
- wire segments 0 -> 360

Commit message: test board for TM1638 and main board finished
Parts:
- removed C2: 10uF, Capacitor_SMD:C_0805_2012Metric, symbol Device:C
- removed U2: TM1638, Package_SO:SOIC-28W_7.5x17.9mm_P1.27mm, symbol beat707:TM1638
- added C11: 10uF, Capacitor_THT:CP_Radial_D6.3mm_P2.50mm, symbol Device:CP
- added U6: TM1638, Package_SO:SOIC-28W_7.5x17.9mm_P1.27mm, symbol beat707:TM1638
- C10: renamed from C1; footprint Capacitor_SMD:C_0805_2012Metric -> Capacitor_THT:C_Disc_D3.0mm_W2.0mm_P2.50mm
- SW10, SW11, SW12, SW13, SW14, SW15, SW16, SW17, SW18, SW19, SW20, SW21, SW22, SW23, SW24, SW25, SW26, SW27, SW28, SW5, SW6, SW7, SW8, SW9: footprint beat707:K2-1103SP-A4SW-04 -> beat707:B3F-through-hole
- renumbered D5 to D10, D6 to D11, D7 to D12, D8 to D13, D13 to D18, D14 to D19, D15 to D20, D16 to D21, D17 to D22, D18 to D23, D19 to D24, D20 to D25, D49 to D54, D50 to D55, D51 to D56, D52 to D57, D1 to D6, D61 to D66, D62 to D67, D63 to D68, D64 to D69, D2 to D7, D65 to D70, D66 to D71, D67 to D72, D68 to D73, D69 to D74, D70 to D75, D71 to D76, D72 to D77, D73 to D78, D74 to D79, D3 to D8, D75 to D80, D76 to D81, D77 to D82, D78 to D83, D79 to D84, D80 to D85, D4 to D9, R35 to R51, R36 to R52, R37 to R53, R38 to R54, R39 to R55, R40 to R56, R41 to R57, R42 to R58, R43 to R59, R44 to R60, R45 to R61, R46 to R62, R47 to R63, R48 to R64, R49 to R65, R50 to R66, R51 to R67, R52 to R68, R53 to R69, R54 to R70, R55 to R71, R56 to R72, R57 to R73, R58 to R74, R59 to R75, R60 to R76, R61 to R77, R62 to R78, R63 to R79, R64 to R80, R65 to R81, R66 to R82, R67 to R83, R68 to R84, U3 to U7, U4 to U8
Connections:
- net labels added: VCC

Commit message: board updated and schematic cleanup
Parts:
- renumbered C10 to C11, C11 to C12
Changed lines of the file:
@@
 	5350 6000 5650 6000
 $Comp
-L power:+5V #PWR051
+L power:+5V #PWR052
 U 1 1 5C9BE63E
 P 4700 3850
-AR Path="/5C65184E/5C9BE63E" Ref="#PWR051"  Part="1"
-AR Path="/5C6557AC/5C9BE63E" Ref="#PWR054"  Part="1"
-AR Path="/5C6559D3/5C9BE63E" Ref="#PWR057"  Part="1"
-F 0 "#PWR057" H 4700 3700 50  0001 C CNN
+AR Path="/5C65184E/5C9BE63E" Ref="#PWR052"  Part="1"
+AR Path="/5C6557AC/5C9BE63E" Ref="#PWR055"  Part="1"
+AR Path="/5C6559D3/5C9BE63E" Ref="#PWR058"  Part="1"
+F 0 "#PWR058" H 4700 3700 50  0001 C CNN
 F 1 "+5V" H 4715 4023 50  0000 C CNN
 F 2 "" H 4700 3850 50  0001 C CNN
@@
 	4700 3850 4700 3900
 $Comp
-L power:GND #PWR052
+L power:GND #PWR053
 U 1 1 5C9D87ED
 P 4700 6550
-AR Path="/5C65184E/5C9D87ED" Ref="#PWR052"  Part="1"
-AR Path="/5C6557AC/5C9D87ED" Ref="#PWR055"  Part="1"
-AR Path="/5C6559D3/5C9D87ED" Ref="#PWR058"  Part="1"
-F 0 "#PWR058" H 4700 6300 50  0001 C CNN
+AR Path="/5C65184E/5C9D87ED" Ref="#PWR053"  Part="1"
+AR Path="/5C6557AC/5C9D87ED" Ref="#PWR056"  Part="1"
+AR Path="/5C6559D3/5C9D87ED" Ref="#PWR059"  Part="1"
+F 0 "#PWR059" H 4700 6300 50  0001 C CNN
 F 1 "GND" H 4705 6377 50  0000 C CNN
 F 2 "" H 4700 6550 50  0001 C CNN
@@
 	4700 6450 4700 6550
 $Comp
-L power:GND #PWR050
+L power:GND #PWR051
 U 1 1 5CA013BE
 P 4350 4350
-AR Path="/5C65184E/5CA013BE" Ref="#PWR050"  Part="1"
-AR Path="/5C6557AC/5CA013BE" Ref="#PWR053"  Part="1"
-AR Path="/5C6559D3/5CA013BE" Ref="#PWR056"  Part="1"
-F 0 "#PWR056" H 4350 4100 50  0001 C CNN
+AR Path="/5C65184E/5CA013BE" Ref="#PWR051"  Part="1"
+AR Path="/5C6557AC/5CA013BE" Ref="#PWR054"  Part="1"
+AR Path="/5C6559D3/5CA013BE" Ref="#PWR057"  Part="1"
+F 0 "#PWR057" H 4350 4100 50  0001 C CNN
 F 1 "GND" H 4355 4177 50  0000 C CNN
 F 2 "" H 4350 4350 50  0001 C CNN
@@
 $EndComp
 $Comp
-L Device:C C10
+L Device:C C11
 U 1 1 5CA0F350
 P 3850 4100
-AR Path="/5C65184E/5CA0F350" Ref="C10"  Part="1"
-AR Path="/5C6557AC/5CA0F350" Ref="C12"  Part="1"
-AR Path="/5C6559D3/5CA0F350" Ref="C14"  Part="1"
-F 0 "C14" H 3965 4146 50  0000 L CNN
+AR Path="/5C65184E/5CA0F350" Ref="C11"  Part="1"
+AR Path="/5C6557AC/5CA0F350" Ref="C13"  Part="1"
+AR Path="/5C6559D3/5CA0F350" Ref="C15"  Part="1"
+F 0 "C15" H 3965 4146 50  0000 L CNN
 F 1 "100nF" H 3965 4055 50  0000 L CNN
 F 2 "Capacitor_THT:C_Disc_D3.0mm_W2.0mm_P2.50mm" H 3888 3950 50  0001 C CNN
@@
 VCC
 $Comp
-L Device:CP C11
+L Device:CP C12
 U 1 1 5C8D67A3
 P 4350 4100
-AR Path="/5C65184E/5C8D67A3" Ref="C11"  Part="1"
-AR Path="/5C6557AC/5C8D67A3" Ref="C13"  Part="1"
-AR Path="/5C6559D3/5C8D67A3" Ref="C15"  Part="1"
-F 0 "C15" H 4375 4200 50  0000 L CNN
+AR Path="/5C65184E/5C8D67A3" Ref="C12"  Part="1"
+AR Path="/5C6557AC/5C8D67A3" Ref="C14"  Part="1"
+AR Path="/5C6559D3/5C8D67A3" Ref="C16"  Part="1"
+F 0 "C16" H 4375 4200 50  0000 L CNN
 F 1 "10uF" H 4375 4000 50  0000 L CNN
 F 2 "Capacitor_THT:CP_Radial_D6.3mm_P2.50mm" H 4388 3950 50  0001 C CNN

Commit message: restored deleted files and added all 3D models
Connections:
- wire segments 360 -> 288
