File: kicad/beat707/fram-test.sch (KiCad schematic (older format))
At the start: 15 parts, among them J1 Conn_01x06_Male, Q1 2N7000, U3 MB85RS2MT, U4 LP2950CZ-3.3G

Commit message: new FRAM test and TM!638 board cleanups
Parts:
- removed C7: 10uF, Capacitor_THT:CP_Radial_D6.3mm_P2.50mm, symbol Device:CP
- removed Q1: 2N7000, Package_TO_SOT_THT:TO-92_Inline, symbol Transistor_FET:2N7000
- removed R5, R7, R8: 3.3k, Resistor_THT:R_Axial_DIN0207_L6.3mm_D2.5mm_P7.62mm_Horizontal, symbol Device:R
- removed R6: 2.2k, Resistor_THT:R_Axial_DIN0207_L6.3mm_D2.5mm_P7.62mm_Horizontal, symbol Device:R
- added H1, H2, H3, H4: MountingHole, MountingHole:MountingHole_2.2mm_M2, symbol Mechanical:MountingHole
- added J2: 3.3V, Connector_PinHeader_2.54mm:PinHeader_1x01_P2.54mm_Vertical, symbol Connector:Conn_01x01_Male
- added J3: GND, Connector_PinHeader_2.54mm:PinHeader_1x01_P2.54mm_Vertical, symbol Connector:Conn_01x01_Male
- added U1, U2, U5, U6: SN74LVC1T45DCK, Package_TO_SOT_SMD:SOT-363_SC-70-6, symbol Logic_LevelTranslator:SN74LVC1T45DCK
- R1, R3: value 2.2k -> 33; footprint Resistor_THT:R_Axial_DIN0207_L6.3mm_D2.5mm_P7.62mm_Horizontal -> Resistor_THT:R_Axial_DIN0207_L6.3mm_D2.5mm_P10.16mm_Horizontal
- R2, R4: value 3.3k -> 33; footprint Resistor_THT:R_Axial_DIN0207_L6.3mm_D2.5mm_P7.62mm_Horizontal -> Resistor_THT:R_Axial_DIN0207_L6.3mm_D2.5mm_P10.16mm_Horizontal
Connections:
- net labels added: FRAM-MISO, FRAM-MOSI
- net labels removed: FRAM-SI, FRAM-SO
- wire segments 62 -> 38
Other:
- note added: "A to B"
- note added: "B to A"
- moved on the sheet: C5, J1
