File: kicad/beat707/beat707.sch (KiCad schematic (older format))
At the start: 89 parts, among them J1 footswitch, J10 free IO, J11 ISP, J12 free IO, J13 free IO, J2 click-out, J3 MIDI-in, J4 MIDI-out, J5 serial debug, J6 +5V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

Commit message: final component placement and routing
Connections:
- net GND: now also C7.2, J8.4 (GND), J8.5 (Shield)
Changed lines of the file:
@@
 	1    0    0    -1
 $EndComp
+$Comp
+L power:GND #PWR?
+U 1 1 5D278F7E
+P 5700 7400
+F 0 "#PWR?" H 5700 7150 50  0001 C CNN
+F 1 "GND" H 5550 7400 50  0000 C CNN
+F 2 "" H 5700 7400 50  0001 C CNN
+F 3 "" H 5700 7400 50  0001 C CNN
+	1    5700 7400
+	1    0    0    -1
+$EndComp
+Connection ~ 5700 7400
 $EndSCHEMATC

Commit message: final routed version
Parts:
- added C19, C20: 1nF, Capacitor_THT:C_Disc_D8.0mm_W5.0mm_P7.50mm, symbol Device:C
- added D16, D17, D18, D19: 1N4148, Diode_THT:D_DO-35_SOD27_P7.62mm_Horizontal, symbol Diode:1N4148
- added J14, J15: free IO, Connector_PinHeader_2.54mm:PinHeader_1x01_P2.54mm_Vertical, symbol Connector:Conn_01x01_Male
- added LOGO1: Logo_Open_Hardware_Small, Symbol:OSHW-Logo_19x20mm_SilkScreen, symbol Graphic:Logo_Open_Hardware_Small
- added R32, R33: 220, Resistor_THT:R_Axial_DIN0207_L6.3mm_D2.5mm_P10.16mm_Horizontal, symbol Device:R
Connections:
- net +5V: now also D16.1 (K), D18.1 (K)
- net GND: now also C19.1, C20.1, D17.2 (A), D19.2 (A)
- net tm1638-clk: now also R33.1
- net tm1638-stb: now also R32.1
- new net: C19.2, D16.2 (A), D17.1 (K), J14.1 (Pin_1), R32.2
- new net: C20.2, D18.2 (A), D19.1 (K), J15.1 (Pin_1), R33.2
Other:
- moved on the sheet: C10, C11, C8, C9, D10, D11, D12, D13, D14, D15, D8, D9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

Commit message: changes for new KiCad version, added panel file, and added documentation
Parts:
- J8: symbol Connector:USB_B -> beat707-rescue:USB_B-Connector
- U3: symbol MCU_Microchip_ATmega:ATmega328-PU -> beat707-rescue:ATmega328-PU-MCU_Microchip_ATmega
Changed lines of the file:
@@
 EESchema Schematic File Version 4
-LIBS:beat707-cache
-EELAYER 29 0
+EELAYER 30 0
 EELAYER END
 $Descr A4 11693 8268
@@
 $EndSheet
 $Comp
-L MCU_Microchip_ATmega:ATmega328-PU U3
+L beat707-rescue:ATmega328-PU-MCU_Microchip_ATmega U3
 U 1 1 5C655D4D
 P 6050 3050
@@
 $EndComp
 $Comp
-L Connector:USB_B J8
+L beat707-rescue:USB_B-Connector J8
 U 1 1 5C655E8B
 P 5800 6800
